Commit message: add missing urdf file

File: urdf/hithand.xacro (robot description, xacro)
@@ -3,4 +3,6 @@
     <xacro:include filename="$(find hithand_description)/urdf/transmission.xacro" />
     <xacro:include filename="$(find hithand_description)/urdf/hithand.gazebo" />
+    <xacro:property name="mu1" value="0.6"/>
+    <xacro:property name="mu2" value="0.6"/>
     <link name="world"/>
     <joint name="fixed" type="fixed">
@@ -53,4 +55,12 @@
                     <cylinder length="0.001" radius="0.001" />
                 </geometry>
+                <surface>
+                  <friction>
+                    <ode>
+                      <mu>${mu1}</mu>
+                      <mu2>${mu2}</mu2>
+                    </ode>
+                  </friction>
+                </surface>
             </collision>
       </link>
@@ -85,4 +95,12 @@
                             <box size="0.03 0.03 0.02" />
                     </geometry>
+                    <surface>
+                      <friction>
+                        <ode>
+                          <mu>${mu1}</mu>
+                          <mu2>${mu2}</mu2>
+                        </ode>
+                      </friction>
+                    </surface>
             </collision>
       </link>
@@ -117,4 +135,12 @@
                             <box size="0.01 0.02 0.02" />
             </geometry>
+            <surface>
+              <friction>
+                <ode>
+                  <mu>${mu1}</mu>
+                  <mu2>${mu2}</mu2>
+                </ode>
+              </friction>
+            </surface>
             </collision>
       </link>
@@ -149,4 +175,12 @@
                             <mesh filename="package://hithand_description/meshes/visual/hit-hand-2-finger-phadist.dae" />
                     </geometry>
+                    <surface>
+                      <friction>
+                        <ode>
+                          <mu>${mu1}</mu>
+                          <mu2>${mu2}</mu2>
+                        </ode>
+                      </friction>
+                    </surface>
             </collision>
       </link>
