Commit message: feat: added entire thumb

File: hithand_description/urdf/hithand.transmission.xacro (robot description, xacro)
@@ -12,5 +12,5 @@
       </actuator>
     </transmission>
-    <!-- <transmission name="tran_${finger_name}_1">
+    <transmission name="tran_${finger_name}_1">
       <type>transmission_interface/SimpleTransmission</type>
       <joint name="Right_${finger_name}_1">
@@ -21,6 +21,5 @@
         <mechanicalReduction>1</mechanicalReduction>
       </actuator>
-    </transmission> -->
-    <!--
+    </transmission>
     <transmission name="tran_${finger_name}_2">
         <type>transmission_interface/SimpleTransmission</type>
@@ -42,5 +41,5 @@
           <mechanicalReduction>1</mechanicalReduction>
         </actuator>
-      </transmission> -->
+      </transmission>
   </xacro:macro>
     <xacro:hithand_transmission finger_name="Thumb">

File: hithand_description/urdf/hithand.xacro (robot description, xacro)
@@ -4,5 +4,8 @@
         <xacro:property name="mu1" value="0.6"/>
         <xacro:property name="mu2" value="0.6"/>
-        <xacro:property name="inertia_mag" value="3"/>
+        <xacro:property name="inertia_mag_0" value="3"/> <!-- should be 5 -->
+        <xacro:property name="inertia_mag_1" value="3"/> <!-- should be 5 -->
+        <xacro:property name="inertia_mag_2" value="3"/> <!-- should be 6 -->
+        <xacro:property name="inertia_mag_3" value="3"/> <!-- should be 6 -->
         <!-- Either attach the Hithand to ths specified world link or that a robot link -->
         <xacro:if value="${not attached}">
@@ -60,14 +63,14 @@
                 <child link="Right_${prefix}_Basecover" />
                 <axis xyz="0 0 1" />
-                <!-- <limit effort="15" lower="-0.261799" upper="0.261799" velocity="3.14"/> -->
-                <limit effort="1000" lower="-1" upper="1" velocity="3.14"/>
+                <limit effort="15" lower="-0.261799" upper="0.261799" velocity="3.14"/>
+                <!-- <limit effort="1000" lower="-1" upper="1" velocity="3.14"/> -->
                 <dynamics damping="0.7" friction="0.5" />
             </joint>
             <link name="Right_${prefix}_Basecover">
                 <inertial>
-                    <origin xyz="0 0 0" rpy="0 0 0" />
+                    <origin xyz="0.02749 0 0" rpy="0 0 0" />
                     <!-- <mass value="0.0176" /> -->
-                    <mass value="0.1"/>
-                    <inertia ixx="1e-${inertia_mag}" ixy="0.0" ixz="0.0" iyy="1e-${inertia_mag}" iyz="0.0" izz="1e-${inertia_mag}" />
+                    <mass value="0.0176"/>
+                    <inertia ixx="2e-${inertia_mag_0}" ixy="0.0" ixz="0.0" iyy="2e-${inertia_mag_0}" iyz="0.0" izz="2e-${inertia_mag_0}" />
                 </inertial>
                 <visual>
@@ -86,5 +89,5 @@
             </link>
             <!-- +++++ Finger joint 1 Phalanx proximalis ++++++ -->
-            <!-- <joint name="Right_${prefix}_1" type="revolute">
+            <joint name="Right_${prefix}_1" type="revolute">
                 <origin xyz="0 0 0 " rpy="1.5708 0 0" />
                 <parent link="Right_${prefix}_Basecover" />
@@ -99,5 +102,5 @@
                             rpy="0 0 0" />
                     <mass value="0.0232" />
-                    <inertia ixx="4e-6" ixy="0.0" ixz="0.0" iyy="4e-6" iyz="0.0" izz="4e-6" />
+                    <inertia ixx="2e-${inertia_mag_1}" ixy="0.0" ixz="0.0" iyy="2e-${inertia_mag_1}" iyz="0.0" izz="2e-${inertia_mag_1}" />
                 </inertial>
                 <visual>
@@ -115,6 +118,6 @@
                     </geometry>
                 </collision>
-            </link> -->
-<!--
+            </link>
+            <!-- +++++ Finger joint 2 Phalanx medialis ++++++ -->
             <joint name="Right_${prefix}_2" type="revolute">
                 <origin xyz="0.055 0 0" rpy="0 0 0" />
@@ -127,7 +130,7 @@
             <link name="Right_${prefix}_Phamed">
                 <inertial>
-                    <origin xyz="0 0 0" rpy="0 0 0" />
-                    <mass value="0.01" />
-                    <inertia ixx="0.0001" ixy="0.0" ixz="0.0" iyy="0.0001" iyz="0.0" izz="0.0001" />
+                    <origin xyz="0.0025 0 0" rpy="0 0 0" />
+                    <mass value="0.0158" />
+                    <inertia ixx="1e-${inertia_mag_2}" ixy="0.0" ixz="0.0" iyy="1e-${inertia_mag_2}" iyz="0.0" izz="1e-${inertia_mag_2}" />
                 </inertial>
                 <visual>
@@ -143,19 +146,20 @@
                         <box size="0.01 0.02 0.02" />
                     </geometry>
-                    <surface>
-                        <friction>
-                            <ode>
-                                <mu>${mu1}</mu>
-                                <mu2>${mu2}</mu2>
-                            </ode>
-                        </friction>
-                    </surface>
                 </collision>
             </link>
+            <!-- +++++ Finger joint 3 Phalanx distalis ++++++ -->
+            <joint name="Right_${prefix}_3" type="revolute">
+                <origin xyz="0.025 0 0" rpy="0 0 -1.57" />
+                <parent link="Right_${prefix}_Phamed" />
+                <child link="Right_${prefix}_Phadist" />
+                <axis xyz="0 0 1" />
+                <limit effort="15" lower="-0.50" upper="1.4" velocity="3.14"/>
+                <dynamics damping="0.7" friction="0.5" />
+            </joint>
             <link name="Right_${prefix}_Phadist">
                 <inertial>
-                    <origin xyz="0 0 0" rpy="0 0 0" />
-                    <mass value="0.01" />
-                    <inertia ixx="0.0001" ixy="0.0" ixz="0.0" iyy="0.0001" iyz="0.0" izz="0.0001" />
+                    <origin xyz="0.003 0 0" rpy="0 0 0" />
+                    <mass value="0.0137" />
+                    <inertia ixx="1e-${inertia_mag_3}" ixy="0.0" ixz="0.0" iyy="1e-${inertia_mag_3}" iyz="0.0" izz="1e-${inertia_mag_3}" />
                 </inertial>
                 <visual>
@@ -171,23 +175,8 @@
                         <mesh filename="package://hithand_description/meshes/visual/hit-hand-2-finger-phadist.dae" />
                     </geometry>
-                    <surface>
-                        <friction>
-                            <ode>
-                                <mu>${mu1}</mu>
-                                <mu2>${mu2}</mu2>
-                            </ode>
-                        </friction>
-                    </surface>
                 </collision>
             </link>
-            <joint name="Right_${prefix}_3" type="revolute">
-                <origin xyz="0.025 0 0" rpy="0 0 -1.57" />
-                <parent link="Right_${prefix}_Phamed" />
-                <child link="Right_${prefix}_Phadist" />
-                <axis xyz="0 0 1" />
-                <limit effort="15" lower="-0.50" upper="1.4" velocity="3.14"/>
-                <dynamics damping="0.7" friction="0.5" />
-            </joint> -->
         </xacro:macro>
+        <!-- #########################FINGER######################## -->
         <!-- END of finger macro -->
         <xacro:finger prefix="Thumb"  >

Commit message: feat: add transm and gazebo config for all joints and links

File: hithand_description/urdf/hithand.transmission.xacro (robot description, xacro)
@@ -45,5 +45,5 @@
     <xacro:hithand_transmission finger_name="Thumb">
     </xacro:hithand_transmission>
-    <!-- <xacro:hithand_transmission finger_name="Index">
+    <xacro:hithand_transmission finger_name="Index">
     </xacro:hithand_transmission>
     <xacro:hithand_transmission finger_name="Middle">
@@ -52,4 +52,4 @@
     </xacro:hithand_transmission>
     <xacro:hithand_transmission finger_name="Little">
-    </xacro:hithand_transmission> -->
+    </xacro:hithand_transmission>
 </robot>

File: hithand_description/urdf/hithand.xacro (robot description, xacro)
@@ -42,5 +42,5 @@
       		    <origin rpy="0 0 0" xyz="0 0 0.05" />
       		    <geometry name="hithand_right_palm_collision">
-        		    <box size="0.1 0.1 0.1" />
+        		    <box size="0.06 0.1 0.07" />
       		    </geometry>
     	    </collision>
@@ -63,4 +63,5 @@
                 <child link="Right_${prefix}_Basecover" />
                 <axis xyz="0 0 1" />
+                <!-- <limit effort="15" lower="-1" upper="1" velocity="3.14"/> -->
                 <limit effort="15" lower="-0.261799" upper="0.261799" velocity="3.14"/>
                 <!-- <limit effort="1000" lower="-1" upper="1" velocity="3.14"/> -->
@@ -94,5 +95,7 @@
                 <child link="Right_${prefix}_Phaprox" />
                 <axis xyz="0 0 1" />
-                <limit effort="15" lower="0.0872665" upper="1.48353" velocity="3.14"/>
+                <!-- <limit effort="15" lower="-1" upper="1" velocity="3.14"/> -->
+                <!-- <limit effort="15" lower="0.0872665" upper="1.48353" velocity="3.14"/> -->
+                <limit effort="15" lower="0" upper="1.48353" velocity="3.14"/>
                 <dynamics damping="0.7" friction="0.5" />
             </joint>
@@ -125,5 +128,7 @@
                 <child link="Right_${prefix}_Phamed" />
                 <axis xyz="0 0 1" />
-                <limit effort="15" lower="0.0872665" upper="1.13446" velocity="3.14"/>
+                <!-- <limit effort="15" lower="-1" upper="1" velocity="3.14"/> -->
+                <!-- <limit effort="15" lower="0.0872665" upper="1.13446" velocity="3.14"/> -->
+                <limit effort="15" lower="0" upper="1.13446" velocity="3.14"/>
                 <dynamics damping="0.7" friction="0.5" />
             </joint>
@@ -154,4 +159,5 @@
                 <child link="Right_${prefix}_Phadist" />
                 <axis xyz="0 0 1" />
+                <!-- <limit effort="15" lower="-1" upper="1" velocity="3.14"/> -->
                 <limit effort="15" lower="-0.50" upper="1.4" velocity="3.14"/>
                 <dynamics damping="0.7" friction="0.5" />
@@ -170,10 +176,10 @@
                     <material name="lightblue"/>
                 </visual>
-                <!-- <collision>
+                <collision>
                     <origin xyz="0 0 0" rpy="0 0 0" />
                     <geometry name='hithand_${prefix}_phadist'>
                         <mesh filename="package://hithand_description/meshes/visual/hit-hand-2-finger-phadist.dae" />
                     </geometry>
-                </collision> -->
+                </collision>
             </link>
         </xacro:macro>
@@ -181,6 +187,22 @@
         <!-- END of finger macro -->
         <xacro:finger prefix="Thumb"  >
-                <origin xyz="0.06217593 0.044372912 0.078734808"
-                        rpy="0.225810 -1.083656 0.411355" />
+            <origin xyz="0.06217593 0.044372912 0.078734808"
+                    rpy="0.225810 -1.083656 0.411355" />
+        </xacro:finger>
+        <xacro:finger prefix="Index"  >
+            <origin xyz="-0.002529881 0.03680013 0.107783545"
+                    rpy="3.054326 -1.570796 0.000000" />
+        </xacro:finger>
+        <xacro:finger prefix="Middle"  >
+            <origin xyz="-0.0037 0.01  0.117783545"
+                    rpy="-3.141593 -1.570796 0.000000" />
+        </xacro:finger>
+        <xacro:finger prefix="Ring"   >
+            <origin xyz="0 -0.01680013 0.11258354"
+                    rpy="-3.054326 -1.570796 0.000000" />
+        </xacro:finger>
+        <xacro:finger prefix="Little"  >
+            <origin xyz="0.000971571 -0.0433963 0.093583545"
+                    rpy="-2.967060 -1.570796 0.000000" />
         </xacro:finger>
     </xacro:macro>
