Commit message: feat: effort control thumb joint 0

File: hithand_description/urdf/hithand.xacro (robot description, xacro)
@@ -1,222 +1,202 @@
-<?xml version="1.0"?>
+<?xml version="1.0" ?>
 <robot xmlns:xacro="http://www.ros.org/wiki/xacro" name="hithand">
-    <xacro:include filename="$(find hithand_description)/urdf/transmission.xacro" />
-    <xacro:include filename="$(find hithand_description)/urdf/hithand.gazebo" />
-    <xacro:property name="mu1" value="0.6"/>
-    <xacro:property name="mu2" value="0.6"/>
-    <link name="world"/>
-    <joint name="fixed" type="fixed">
-        <parent link="world"/>
-        <child link="base_link"/>
-    </joint>
-    <link name="base_link">
-  	<inertial>
-      		<origin xyz="0.0 0.0 0.0"
-        		rpy="0 0 0" />
-      		<mass value="1.0"/>
-      		<inertia ixx="1.0" ixy="0.0" ixz="0.0" iyy="1.0" iyz="0.0" izz="1.0" />
-    	</inertial>
-   	<visual>
-      		<origin rpy="0 0 0" xyz="0 0 0" />
-      		<geometry>
-        		<mesh filename="package://hithand_description/meshes/visual/hit-hand-2-palm-right.dae"/>
-      		</geometry>
-      		<material name="grey" />
-    	</visual>
-    	<collision>
-      		<origin rpy="0 0 0" xyz="0 0 0" />
-      		<geometry name="hithand_right_palm_collision">
-        		<cylinder length="0.001" radius="0.001" />
-      		</geometry>
-    	</collision>
-  </link>
-    <xacro:macro name="finger" params="prefix *transform_palm2finger">
-        <!-- #########################fINGER######################## -->
-        <link name="Right_${prefix}_Basecover">
-            <inertial>
-                <origin xyz="0 0 0"
-                    rpy="0 0 0" />
-                <mass value="1.0" />
-                <inertia ixx="1.0" ixy="0.0" ixz="0.0" iyy="1.0" iyz="0.0" izz="1.0" />
-            </inertial>
-            <visual>
-                <origin xyz="0 0 0"
-                    rpy="0 0 0" />
-                <geometry>
-                <!-- <mesh filename="file://$(arg meshDirectory)visual/hit-hand-2-finger-basecover.dae" /> -->
-                <mesh filename="package://hithand_description/meshes/visual/hit-hand-2-finger-basecover.dae"/>
-                </geometry>
-            <material name="white"/>
-            </visual>
-            <collision>
-                <origin xyz="0 0 0"
-                    rpy="0 0 0" />
-                <geometry name='hithand_${prefix}_base_cover'>
-                    <cylinder length="0.001" radius="0.001" />
-                </geometry>
-                <surface>
-                  <friction>
-                    <ode>
-                      <mu>${mu1}</mu>
-                      <mu2>${mu2}</mu2>
-                    </ode>
-                  </friction>
-                </surface>
-            </collision>
-      </link>
-      <joint name="Right_${prefix}_1"
-        type="revolute">
-            <!-- joint origin in parent link frame -->
-            <xacro:insert_block name="transform_palm2finger" />
-            <parent link="base_link" />
-            <child link="Right_${prefix}_Basecover" />
-        <axis xyz="0 0 1" />
-        <limit effort="1000" lower="-0.50" upper="1.4" velocity="3.14"/>
-          <dynamics damping="0.7" friction="0.5" />
-      </joint>
-      <link name="Right_${prefix}_Phoaprox">
-            <inertial>
-                    <origin xyz="0.06217593 0.044372912 0.078734808"
-                            rpy="0.225810 -1.083656 0.411355" />
-                    <mass value="1.0" />
-                    <inertia ixx="1.0" ixy="0.0" ixz="0.0" iyy="1.0" iyz="0.0" izz="1.0" />
-            </inertial>
-            <visual>
-                    <origin xyz="0 0 0"
+    <xacro:macro name="hithand" params="attached:='false' parent:='' ns:='' rpy:='0 0 0' xyz:='0 0 0' ">
+        <xacro:property name="mu1" value="0.6"/>
+        <xacro:property name="mu2" value="0.6"/>
+        <xacro:property name="inertia_mag" value="3"/>
+        <!-- Either attach the Hithand to ths specified world link or that a robot link -->
+        <xacro:if value="${not attached}">
+        <link name="world"/>
+            <joint name="fixed" type="fixed">
+                <parent link="world"/>
+                <child link="base_link_hithand"/>
+                <origin xyz="0 0 0.1" rpy="0 0 0"/>
+            </joint>
+        </xacro:if>
+        <xacro:if value="${attached}">
+            <joint name="${ns}_hithand_joint" type="fixed">
+                <parent link="${parent}"/>
+                <child link="base_link_hithand"/>
+                <origin xyz="${xyz}" rpy="${rpy}"/>
+            </joint>
+        </xacro:if>
+        <!-- ++++ Define all the links and joints ++++ -->
+        <!-- Starting from the base -->
+        <link name="base_link_hithand">
+  	        <inertial>
+      		    <origin xyz="0.0 0.0 0.05" rpy="0 0 0" />
+      		    <mass value="1"/>
+      		    <inertia ixx="1e-3" ixy="0.0" ixz="0.0" iyy="1e-3" iyz="0.0" izz="1e-3" />
+    	    </inertial>
+   	        <visual>
+      		    <origin rpy="0 0 0" xyz="0 0 0" />
+      		    <geometry>
+        		    <mesh filename="package://hithand_description/meshes/visual/hit-hand-2-palm-right.dae"/>
+      		    </geometry>
+      		    <material name="grey" />
+    	    </visual>
+    	    <collision>
+      		    <origin rpy="0 0 0" xyz="0 0 0.05" />
+      		    <geometry name="hithand_right_palm_collision">
+        		    <box size="0.1 0.1 0.1" />
+      		    </geometry>
+    	    </collision>
+        </link>
+        <!-- Add a virtual palm link, just to get the transform of this point via TF for grasping -->
+        <joint name="$hithand_palm_joint" type="fixed">
+            <parent link="base_link_hithand"/>
+            <child link="palm_link_hithand"/>
+            <origin xyz="0.02 0 0.06" rpy="-0.15 -1.15 0"/>
+        </joint>
+        <link name="palm_link_hithand"/>
+        <!-- #########################FINGER######################## -->
+        <!-- Define the fingers in a macro (all fingers are equal) -->
+        <xacro:macro name="finger" params="prefix *transform_palm2finger">
+            <!-- +++++ Finger base joint 0 ++++++ -->
+            <joint name="Right_${prefix}_0" type="revolute">
+                <!-- joint origin in parent link frame -->
+                <xacro:insert_block name="transform_palm2finger" />
+                <parent link="base_link_hithand" />
+                <child link="Right_${prefix}_Basecover" />
+                <axis xyz="0 0 1" />
+                <!-- <limit effort="15" lower="-0.261799" upper="0.261799" velocity="3.14"/> -->
+                <limit effort="1000" lower="-1" upper="1" velocity="3.14"/>
+                <dynamics damping="0.7" friction="0.5" />
+            </joint>
+            <link name="Right_${prefix}_Basecover">
+                <inertial>
+                    <origin xyz="0 0 0" rpy="0 0 0" />
+                    <!-- <mass value="0.0176" /> -->
+                    <mass value="0.1"/>
+                    <inertia ixx="1e-${inertia_mag}" ixy="0.0" ixz="0.0" iyy="1e-${inertia_mag}" iyz="0.0" izz="1e-${inertia_mag}" />
+                </inertial>
+                <visual>
+                    <origin xyz="0 0 0" rpy="0 0 0" />
+                    <geometry>
+                        <mesh filename="package://hithand_description/meshes/visual/hit-hand-2-finger-basecover.dae"/>
+                    </geometry>
+                    <material name="white"/>
+                </visual>
+                <collision>
+                    <origin xyz="0 0 0" rpy="0 0 0" />
+                    <geometry name='hithand_${prefix}_base_cover'>
+                        <cylinder length="0.001" radius="0.001" />
+                    </geometry>
+                </collision>
+            </link>
+            <!-- +++++ Finger joint 1 Phalanx proximalis ++++++ -->
+            <!-- <joint name="Right_${prefix}_1" type="revolute">
+                <origin xyz="0 0 0 " rpy="1.5708 0 0" />
+                <parent link="Right_${prefix}_Basecover" />
+                <child link="Right_${prefix}_Phaprox" />
+                <axis xyz="0 0 1" />
+                <limit effort="15" lower="0.0872665" upper="1.48353" velocity="3.14"/>
+                <dynamics damping="0.7" friction="0.5" />
+            </joint>
+            <link name="Right_${prefix}_Phaprox">
+                <inertial>
+                    <origin xyz="0.02749 0 0"
                             rpy="0 0 0" />
-                    <geometry>
-                            <mesh filename="package://hithand_description/meshes/visual/hit-hand-2-finger-phaprox.dae" />
-                    </geometry>
-            <material name="lightblue"/>
-            </visual>
-            <collision>
+                    <mass value="0.0232" />
+                    <inertia ixx="4e-6" ixy="0.0" ixz="0.0" iyy="4e-6" iyz="0.0" izz="4e-6" />
+                </inertial>
+                <visual>
+                    <origin xyz="0 0 0" rpy="0 0 0" />
+                        <geometry>
+                                <mesh filename="package://hithand_description/meshes/visual/hit-hand-2-finger-phaprox.dae" />
+                        </geometry>
+                    <material name="lightblue"/>
+                </visual>
+                <collision>
                     <origin xyz="0.03 0 0"
                             rpy="0 0 0" />
-                    <geometry name='hithand_${prefix}_phoarpox'>
-                            <box size="0.03 0.03 0.02" />
+                    <geometry name='hithand_${prefix}_phaprox'>
+                        <box size="0.03 0.03 0.02" />
+                    </geometry>
+                </collision>
+            </link> -->
+<!--
+            <joint name="Right_${prefix}_2" type="revolute">
+                <origin xyz="0.055 0 0" rpy="0 0 0" />
+                <parent link="Right_${prefix}_Phaprox" />
+                <child link="Right_${prefix}_Phamed" />
+                <axis xyz="0 0 1" />
+                <limit effort="15" lower="0.0872665" upper="1.13446" velocity="3.14"/>
+                <dynamics damping="0.7" friction="0.5" />
+            </joint>
+            <link name="Right_${prefix}_Phamed">
+                <inertial>
+                    <origin xyz="0 0 0" rpy="0 0 0" />
+                    <mass value="0.01" />
+                    <inertia ixx="0.0001" ixy="0.0" ixz="0.0" iyy="0.0001" iyz="0.0" izz="0.0001" />
+                </inertial>
+                <visual>
+                    <origin xyz="0 0 0" rpy="0 0 0" />
+                    <geometry>
+                        <mesh filename="package://hithand_description/meshes/visual/hit-hand-2-finger-phamed.dae" />
+                    </geometry>
+                    <material name="white"/>
+                </visual>
+                <collision>
+                    <origin xyz="0.01 0 0" rpy="0 0 0" />
+                    <geometry name='hithand_${prefix}_phamed'>
+                        <box size="0.01 0.02 0.02" />
                     </geometry>
                     <surface>
-                      <friction>
-                        <ode>
-                          <mu>${mu1}</mu>
-                          <mu2>${mu2}</mu2>
-                        </ode>
-                      </friction>
+                        <friction>
+                            <ode>
+                                <mu>${mu1}</mu>
+                                <mu2>${mu2}</mu2>
+                            </ode>
+                        </friction>
                     </surface>
-            </collision>
-      </link>
-      <joint name="Right_${prefix}_2"
-        type="revolute">
-            <origin xyz="0 0 0 "
-                    rpy="1.5708 0 0" />
-            <parent link="Right_${prefix}_Basecover" />
-            <child link="Right_${prefix}_Phoaprox" />
-            <axis xyz="0 0 1" />
-            <limit effort="1000" lower="-0.50" upper="1.4" velocity="3.14"/>
-            <dynamics damping="0.7" friction="0.5" />
-      </joint>
-      <link name="Right_${prefix}_Phamed">
-            <inertial>
-                    <origin xyz="0 0 0"
-                            rpy="0 0 0" />
-                    <mass value="1.0" />
-                    <inertia ixx="1.0" ixy="0.0" ixz="0.0" iyy="1.0" iyz="0.0" izz="1.0" />
-            </inertial>
-            <visual>
-                    <origin xyz="0 0 0"
-                            rpy="0 0 0" />
+                </collision>
+            </link>
+            <link name="Right_${prefix}_Phadist">
+                <inertial>
+                    <origin xyz="0 0 0" rpy="0 0 0" />
+                    <mass value="0.01" />
+                    <inertia ixx="0.0001" ixy="0.0" ixz="0.0" iyy="0.0001" iyz="0.0" izz="0.0001" />
+                </inertial>
+                <visual>
+                    <origin xyz="0 0 0" rpy="0 0 0" />
                     <geometry>
-                <mesh filename="package://hithand_description/meshes/visual/hit-hand-2-finger-phamed.dae" />
-                    </geometry>
-            <material name="white"/>
-            </visual>
-            <collision>
-                    <origin xyz="0.01 0 0"
-                            rpy="0 0 0" />
-                    <geometry name='hithand_${prefix}_phamed'>
-                            <box size="0.01 0.02 0.02" />
-            </geometry>
-            <surface>
-              <friction>
-                <ode>
-                  <mu>${mu1}</mu>
-                  <mu2>${mu2}</mu2>
-                </ode>
-              </friction>
-            </surface>
-            </collision>
-      </link>
-      <joint name="Right_${prefix}_3"
-        type="revolute">
-            <origin xyz="0.055 0 0"
-                    rpy="0 0 0" />
-            <parent link="Right_${prefix}_Phoaprox" />
-            <child link="Right_${prefix}_Phamed" />
-            <axis xyz="0 0 1" />
-            <limit effort="1000" lower="-0.50" upper="1.4" velocity="3.14"/>
-          <dynamics damping="0.7" friction="0.5" />
-      </joint>
-      <link name="Right_${prefix}_Phadist">
-            <inertial>
-                    <origin xyz="0 0 0"
-                            rpy="0 0 0" />
-                    <mass value="1.0" />
-                    <inertia ixx="1.0" ixy="0.0" ixz="0.0" iyy="1.0" iyz="0.0" izz="1.0" />
-            </inertial>
-            <visual>
-                    <origin xyz="0 0 0"
-                            rpy="0 0 0" />
-                    <geometry>
-                            <mesh filename="package://hithand_description/meshes/visual/hit-hand-2-finger-phadist.dae" />
+                        <mesh filename="package://hithand_description/meshes/visual/hit-hand-2-finger-phadist.dae" />
                     </geometry>
                     <material name="lightblue"/>
-            </visual>
-            <collision>
-                    <origin xyz="0 0 0"
-                            rpy="0 0 0" />
+                </visual>
+                <collision>
+                    <origin xyz="0 0 0" rpy="0 0 0" />
                     <geometry name='hithand_${prefix}_phadist'>
-                            <mesh filename="package://hithand_description/meshes/visual/hit-hand-2-finger-phadist.dae" />
+                        <mesh filename="package://hithand_description/meshes/visual/hit-hand-2-finger-phadist.dae" />
                     </geometry>
                     <surface>
-                      <friction>
-                        <ode>
-                          <mu>${mu1}</mu>
-                          <mu2>${mu2}</mu2>
-                        </ode>
-                      </friction>
+                        <friction>
+                            <ode>
+                                <mu>${mu1}</mu>
+                                <mu2>${mu2}</mu2>
+                            </ode>
+                        </friction>
                     </surface>
-            </collision>
-      </link>
-      <joint name="Right_${prefix}_4"
-        type="revolute">
-            <origin xyz="0.025 0 0"
-                    rpy="0 0 -1.57" />
-            <parent link="Right_${prefix}_Phamed" />
-            <child link="Right_${prefix}_Phadist" />
-            <axis xyz="0 0 1" />
-            <limit effort="1000" lower="-0.50" upper="1.4" velocity="3.14"/>
-          <dynamics damping="0.7" friction="0.5" />
-      </joint>
+                </collision>
+            </link>
+            <joint name="Right_${prefix}_3" type="revolute">
+                <origin xyz="0.025 0 0" rpy="0 0 -1.57" />
+                <parent link="Right_${prefix}_Phamed" />
+                <child link="Right_${prefix}_Phadist" />
+                <axis xyz="0 0 1" />
+                <limit effort="15" lower="-0.50" upper="1.4" velocity="3.14"/>
+                <dynamics damping="0.7" friction="0.5" />
+            </joint> -->
+        </xacro:macro>
+        <!-- END of finger macro -->
+        <xacro:finger prefix="Thumb"  >
+                <origin xyz="0.06217593 0.044372912 0.078734808"
+                        rpy="0.225810 -1.083656 0.411355" />
+        </xacro:finger>
     </xacro:macro>
-+
-    <xacro:finger prefix="Thumb"  >
-            <origin xyz="0.06217593 0.044372912 0.078734808"
-            rpy="0.225810 -1.083656 0.411355" />
-    </xacro:finger>
-    <xacro:finger prefix="Index"  >
-        <origin xyz="-0.002529881 0.03680013 0.107783545"
-      		rpy="3.054326 -1.570796 0.000000" />
-    </xacro:finger>
-    <xacro:finger prefix="Middle"  >
-            <origin xyz="-0.0037 0.01  0.117783545"
-      		rpy="-3.141593 -1.570796 0.000000" />
-    </xacro:finger>
-    <xacro:finger prefix="Ring"   >
-            <origin xyz="0 -0.01680013 0.11258354"
-            rpy="-3.054326 -1.570796 0.000000" />
-    </xacro:finger>
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
Commit message: chore: changed inertia magnitude and collision

File: hithand_description/urdf/hithand.xacro (robot description, xacro)
@@ -4,8 +4,8 @@
         <xacro:property name="mu1" value="0.6"/>
         <xacro:property name="mu2" value="0.6"/>
-        <xacro:property name="inertia_mag_0" value="3"/> <!-- should be 5 -->
-        <xacro:property name="inertia_mag_1" value="3"/> <!-- should be 5 -->
-        <xacro:property name="inertia_mag_2" value="3"/> <!-- should be 6 -->
-        <xacro:property name="inertia_mag_3" value="3"/> <!-- should be 6 -->
+        <xacro:property name="inertia_mag_0" value="6"/> <!-- should be 5 -->
+        <xacro:property name="inertia_mag_1" value="6"/> <!-- should be 5 -->
+        <xacro:property name="inertia_mag_2" value="6"/> <!-- should be 6 -->
+        <xacro:property name="inertia_mag_3" value="6"/> <!-- should be 6 -->
         <!-- Either attach the Hithand to ths specified world link or that a robot link -->
         <xacro:if value="${not attached}">
@@ -170,10 +170,10 @@
                     <material name="lightblue"/>
                 </visual>
-                <collision>
+                <!-- <collision>
                     <origin xyz="0 0 0" rpy="0 0 0" />
                     <geometry name='hithand_${prefix}_phadist'>
                         <mesh filename="package://hithand_description/meshes/visual/hit-hand-2-finger-phadist.dae" />
                     </geometry>
-                </collision>
+                </collision> -->
             </link>
         </xacro:macro>
