Commit message: chore: remove unnecessary lines

File: hithand_description/urdf/hithand.xacro (robot description, xacro)
@@ -8,5 +8,5 @@
         <xacro:property name="inertia_mag_2" value="6"/> <!-- should be 6 -->
         <xacro:property name="inertia_mag_3" value="6"/> <!-- should be 6 -->
-        <!-- Either attach the Hithand to ths specified world link or that a robot link -->
+        <!-- Either attach the Hithand to the then here defined world link or attach to given robot link which itself defines the world frame -->
         <xacro:if value="${not attached}">
         <link name="world"/>
@@ -35,16 +35,21 @@
       		    <origin rpy="0 0 0" xyz="0 0 0" />
       		    <geometry>
-        		    <mesh filename="package://hithand_description/meshes/visual/hit-hand-2-palm-right.dae"/>
+        		    <mesh filename="package://hithand_description/meshes/visual/handhit-hand-2-palm-right.dae"/>
       		    </geometry>
       		    <material name="grey" />
     	    </visual>
     	    <collision>
-      		    <origin rpy="0 0 0" xyz="0 0 0.05" />
+      		    <!-- <origin rpy="0 0 0" xyz="0 0 0.05" />
       		    <geometry name="hithand_right_palm_collision">
         		    <box size="0.06 0.1 0.07" />
+      		    </geometry> -->
+                <origin rpy="0 0 0" xyz="0 0 0" />
+      		    <geometry>
+        		    <mesh filename="package://hithand_description/meshes/collision/hit-hand-2-palm-right.dae"/>
       		    </geometry>
     	    </collision>
         </link>
-        <!-- Add a virtual palm link, just to get the transform of this point via TF for grasping -->
+        <!-- Add a virtual palm link to get the transform of this point via TF for grasping (we align this frame with
+        a normal of an object point cloud.) -->
         <joint name="$hithand_palm_joint" type="fixed">
             <parent link="base_link_hithand"/>
@@ -63,7 +68,5 @@
                 <child link="Right_${prefix}_Basecover" />
                 <axis xyz="0 0 1" />
-                <!-- <limit effort="15" lower="-1" upper="1" velocity="3.14"/> -->
                 <limit effort="15" lower="-0.261799" upper="0.261799" velocity="3.14"/>
-                <!-- <limit effort="1000" lower="-1" upper="1" velocity="3.14"/> -->
                 <dynamics damping="0.7" friction="0.5" />
             </joint>
@@ -89,5 +92,5 @@
                 </collision>
             </link>
-            <!-- +++++ Finger joint 1 Phalanx proximalis ++++++ -->
+            <!-- +++++ Finger joint 1, Link: Phalanx proximalis ++++++ -->
             <joint name="Right_${prefix}_1" type="revolute">
                 <origin xyz="0 0 0 " rpy="1.5708 0 0" />
@@ -95,6 +98,4 @@
                 <child link="Right_${prefix}_Phaprox" />
                 <axis xyz="0 0 1" />
-                <!-- <limit effort="15" lower="-1" upper="1" velocity="3.14"/> -->
-                <!-- <limit effort="15" lower="0.0872665" upper="1.48353" velocity="3.14"/> -->
                 <limit effort="15" lower="0" upper="1.48353" velocity="3.14"/>
                 <dynamics damping="0.7" friction="0.5" />
@@ -115,9 +116,13 @@
                 </visual>
                 <collision>
-                    <origin xyz="0.03 0 0"
+                    <!-- <origin xyz="0.03 0 0"
                             rpy="0 0 0" />
                     <geometry name='hithand_${prefix}_phaprox'>
                         <box size="0.03 0.03 0.02" />
-                    </geometry>
+                    </geometry> -->
+                    <origin xyz="0 0 0" rpy="0 0 0" />
+                        <geometry>
+                                <mesh filename="package://hithand_description/meshes/collision/finger/hit-hand-2-finger-phaprox.dae" />
+                        </geometry>
                 </collision>
             </link>
@@ -128,6 +133,4 @@
                 <child link="Right_${prefix}_Phamed" />
                 <axis xyz="0 0 1" />
-                <!-- <limit effort="15" lower="-1" upper="1" velocity="3.14"/> -->
-                <!-- <limit effort="15" lower="0.0872665" upper="1.13446" velocity="3.14"/> -->
                 <limit effort="15" lower="0" upper="1.13446" velocity="3.14"/>
                 <dynamics damping="0.7" friction="0.5" />
@@ -147,8 +150,12 @@
                 </visual>
                 <collision>
-                    <origin xyz="0.01 0 0" rpy="0 0 0" />
+                    <!-- <origin xyz="0.01 0 0" rpy="0 0 0" />
                     <geometry name='hithand_${prefix}_phamed'>
                         <box size="0.01 0.02 0.02" />
-                    </geometry>
+                    </geometry> -->
+                    <origin xyz="0 0 0" rpy="0 0 0" />
+                        <geometry>
+                                <mesh filename="package://hithand_description/meshes/collision/finger/hit-hand-2-finger-phamed.dae" />
+                        </geometry>
                 </collision>
             </link>
@@ -177,8 +184,12 @@
                 </visual>
                 <collision>
-                    <origin xyz="0 0 0" rpy="0 0 0" />
+                    <!-- <origin xyz="0 0.01 0" rpy="0 0 0" />
                     <geometry name='hithand_${prefix}_phadist'>
-                        <mesh filename="package://hithand_description/meshes/visual/hit-hand-2-finger-phadist.dae" />
-                    </geometry>
+                        <box size="0.02 0.035 0.02" />
+                    </geometry> -->
+                    <origin xyz="0 0 0" rpy="0 0 0" />
+                        <geometry>
+                                <mesh filename="package://hithand_description/meshes/collision/finger/hit-hand-2-finger-phadist.dae" />
+                        </geometry>
                 </collision>
             </link>

Commit message: feat: added hithand dynamic parameters based on meshlab

File: hithand_description/urdf/hithand.xacro (robot description, xacro)
@@ -28,7 +28,7 @@
         <link name="base_link_hithand">
   	        <inertial>
-      		    <origin xyz="0.0 0.0 0.05" rpy="0 0 0" />
-      		    <mass value="1"/>
-      		    <inertia ixx="1e-3" ixy="0.0" ixz="0.0" iyy="1e-3" iyz="0.0" izz="1e-3" />
+      		    <origin xyz="0.0112 0.0 0.0566" rpy="0 0 0" />
+      		    <mass value="1.1485"/>
+      		    <inertia ixx="2.2458e-3" ixy="2.7421e-4" ixz="1.6e-5" iyy="2.2203e-3" iyz="6.37e-5" izz="1.9003e-3" />
     	    </inertial>
    	        <visual>
@@ -76,5 +76,5 @@
                     <!-- <mass value="0.0176" /> -->
                     <mass value="0.0176"/>
-                    <inertia ixx="2e-${inertia_mag_0}" ixy="0.0" ixz="0.0" iyy="2e-${inertia_mag_0}" iyz="0.0" izz="2e-${inertia_mag_0}" />
+                    <inertia ixx="1.3450e-6" ixy="0.0" ixz="1.8183e-7" iyy="1.9874e-6" iyz="0.0" izz="1.0419e-6" />
                 </inertial>
                 <visual>
@@ -103,8 +103,8 @@
             <link name="Right_${prefix}_Phaprox">
                 <inertial>
-                    <origin xyz="0.02749 0 0"
+                    <origin xyz="0.03076 0.00297 0"
                             rpy="0 0 0" />
                     <mass value="0.0232" />
-                    <inertia ixx="2e-${inertia_mag_1}" ixy="0.0" ixz="0.0" iyy="2e-${inertia_mag_1}" iyz="0.0" izz="2e-${inertia_mag_1}" />
+                    <inertia ixx="2.5326e-6" ixy="9.2551e-7" ixz="4.0954e-8" iyy="6.9625e-6" iyz="0.0" izz="7.9108e-6" />
                 </inertial>
                 <visual>
@@ -138,7 +138,7 @@
             <link name="Right_${prefix}_Phamed">
                 <inertial>
-                    <origin xyz="0.0025 0 0" rpy="0 0 0" />
+                    <origin xyz="0.0097 -0.00036 0" rpy="0 0 0" />
                     <mass value="0.0158" />
-                    <inertia ixx="1e-${inertia_mag_2}" ixy="0.0" ixz="0.0" iyy="1e-${inertia_mag_2}" iyz="0.0" izz="1e-${inertia_mag_2}" />
+                    <inertia ixx="1.1852e-6" ixy="2.8845e-8" ixz="6.1323e-9" iyy="2.4460e-6" iyz="2.4541e-9" izz="2.6537e-6" />
                 </inertial>
                 <visual>
@@ -172,7 +172,7 @@
             <link name="Right_${prefix}_Phadist">
                 <inertial>
-                    <origin xyz="0.003 0 0" rpy="0 0 0" />
+                    <origin xyz="0.00072 0.00717 0.0" rpy="0 0 0" />
                     <mass value="0.0137" />
-                    <inertia ixx="1e-${inertia_mag_3}" ixy="0.0" ixz="0.0" iyy="1e-${inertia_mag_3}" iyz="0.0" izz="1e-${inertia_mag_3}" />
+                    <inertia ixx="1.5519e-6" ixy="0.0" ixz="0.0" iyy="8.2972e-7" iyz="0.0" izz="1.5788e-6" />
                 </inertial>
                 <visual>

Commit message: perf: model friction of the hithand

File: hithand_description/urdf/hithand.xacro (robot description, xacro)
@@ -35,5 +35,5 @@
       		    <origin rpy="0 0 0" xyz="0 0 0" />
       		    <geometry>
-        		    <mesh filename="package://hithand_description/meshes/visual/handhit-hand-2-palm-right.dae"/>
+        		    <mesh filename="package://hithand_description/meshes/visual/hit-hand-2-palm-right.dae"/>
       		    </geometry>
       		    <material name="grey" />
@@ -48,4 +48,12 @@
         		    <mesh filename="package://hithand_description/meshes/collision/hit-hand-2-palm-right.dae"/>
       		    </geometry>
+                <surface>
+                    <friction>
+                        <ode>
+                            <mu>0.8</mu>
+                            <mu2>0.8</mu2>
+                        </ode>
+                    </friction>
+                </surface>
     	    </collision>
         </link>
@@ -81,5 +89,5 @@
                     <origin xyz="0 0 0" rpy="0 0 0" />
                     <geometry>
-                        <mesh filename="package://hithand_description/meshes/visual/hit-hand-2-finger-basecover.dae"/>
+                        <mesh filename="package://hithand_description/meshes/visual/finger/hit-hand-2-finger-basecover.dae"/>
                     </geometry>
                     <material name="white"/>
@@ -111,5 +119,5 @@
                     <origin xyz="0 0 0" rpy="0 0 0" />
                         <geometry>
-                                <mesh filename="package://hithand_description/meshes/visual/hit-hand-2-finger-phaprox.dae" />
+                                <mesh filename="package://hithand_description/meshes/visual/finger/hit-hand-2-finger-phaprox.dae" />
                         </geometry>
                     <material name="lightblue"/>
@@ -125,4 +133,12 @@
                                 <mesh filename="package://hithand_description/meshes/collision/finger/hit-hand-2-finger-phaprox.dae" />
                         </geometry>
+                    <surface>
+                        <friction>
+                            <ode>
+                                <mu>0.8</mu>
+                                <mu2>0.8</mu2>
+                            </ode>
+                        </friction>
+                    </surface>
                 </collision>
             </link>
@@ -145,5 +161,5 @@
                     <origin xyz="0 0 0" rpy="0 0 0" />
                     <geometry>
-                        <mesh filename="package://hithand_description/meshes/visual/hit-hand-2-finger-phamed.dae" />
+                        <mesh filename="package://hithand_description/meshes/visual/finger/hit-hand-2-finger-phamed.dae" />
                     </geometry>
                     <material name="white"/>
@@ -158,9 +174,17 @@
                                 <mesh filename="package://hithand_description/meshes/collision/finger/hit-hand-2-finger-phamed.dae" />
                         </geometry>
+                    <surface>
+                        <friction>
+                            <ode>
+                                <mu>0.6</mu>
+                                <mu2>0.6</mu2>
+                            </ode>
+                        </friction>
+                    </surface>
                 </collision>
             </link>
             <!-- +++++ Finger joint 3 Phalanx distalis ++++++ -->
             <joint name="Right_${prefix}_3" type="revolute">
-                <origin xyz="0.025 0 0" rpy="0 0 -1.57" />
+                <origin xyz="0.025 0 0" rpy="0 0 -1.570796" />
                 <parent link="Right_${prefix}_Phamed" />
                 <child link="Right_${prefix}_Phadist" />
@@ -179,5 +203,5 @@
                     <origin xyz="0 0 0" rpy="0 0 0" />
                     <geometry>
-                        <mesh filename="package://hithand_description/meshes/visual/hit-hand-2-finger-phadist.dae" />
+                        <mesh filename="package://hithand_description/meshes/visual/finger/hit-hand-2-finger-phadist.dae" />
                     </geometry>
                     <material name="lightblue"/>
@@ -192,4 +216,12 @@
                                 <mesh filename="package://hithand_description/meshes/collision/finger/hit-hand-2-finger-phadist.dae" />
                         </geometry>
+                    <surface>
+                        <friction>
+                            <ode>
+                                <mu>0.8</mu>
+                                <mu2>0.8</mu2>
+                            </ode>
+                        </friction>
+                    </surface>
                 </collision>
             </link>

Commit message: fix: increase joint damping to 10 and remove joint friction

File: hithand_description/urdf/hithand.xacro (robot description, xacro)
@@ -30,5 +30,6 @@
       		    <origin xyz="0.0112 0.0 0.0566" rpy="0 0 0" />
       		    <mass value="1.1485"/>
-      		    <inertia ixx="2.2458e-3" ixy="2.7421e-4" ixz="1.6e-5" iyy="2.2203e-3" iyz="6.37e-5" izz="1.9003e-3" />
+      		    <inertia ixx="2.2458e-3" ixy="-2.7421e-4" ixz="1.6e-5" iyy="2.2203e-3" iyz="-6.37e-5" izz="1.9003e-3" />
+                <!-- <inertia ixx="2.2458e-4" ixy="0" ixz="0" iyy="2.2203e-4" iyz="0" izz="1.9003e-4" /> -->
     	    </inertial>
    	        <visual>
@@ -60,5 +61,5 @@
         <!-- Add a virtual palm link to get the transform of this point via TF for grasping (we align this frame with
         a normal of an object point cloud.) -->
-        <joint name="$hithand_palm_joint" type="fixed">
+        <joint name="hithand_palm_joint" type="fixed">
             <parent link="base_link_hithand"/>
             <child link="palm_link_hithand"/>
@@ -68,4 +69,5 @@
         <!-- #########################FINGER######################## -->
         <!-- Define the fingers in a macro (all fingers are equal) -->
+        <!-- Joint limits set according to this: https://github.com/Qianboy/hithand_ros/blob/master/hithand_description/parameter.pdf -->
         <xacro:macro name="finger" params="prefix *transform_palm2finger">
             <!-- +++++ Finger base joint 0 ++++++ -->
@@ -77,5 +79,6 @@
                 <axis xyz="0 0 1" />
                 <limit effort="15" lower="-0.261799" upper="0.261799" velocity="3.14"/>
-                <dynamics damping="0.7" friction="0.5" />
+                <!-- <dynamics damping="0.7" friction="0.5" /> -->
+                <dynamics damping="10" friction="0" />
             </joint>
             <link name="Right_${prefix}_Basecover">
@@ -84,5 +87,6 @@
                     <!-- <mass value="0.0176" /> -->
                     <mass value="0.0176"/>
-                    <inertia ixx="1.3450e-6" ixy="0.0" ixz="1.8183e-7" iyy="1.9874e-6" iyz="0.0" izz="1.0419e-6" />
+                    <inertia ixx="1.3450e-6" ixy="0.0" ixz="-1.8183e-7" iyy="1.9874e-6" iyz="0.0" izz="1.0419e-6" />
+                    <!-- <inertia ixx="1.3450e-6" ixy="0.0" ixz="0" iyy="1.9874e-6" iyz="0.0" izz="1.0419e-6" /> -->
                 </inertial>
                 <visual>
@@ -106,6 +110,8 @@
                 <child link="Right_${prefix}_Phaprox" />
                 <axis xyz="0 0 1" />
-                <limit effort="15" lower="0" upper="1.48353" velocity="3.14"/>
-                <dynamics damping="0.7" friction="0.5" />
+                <limit effort="15" lower="0.0872665" upper="1.48353" velocity="3.14"/>
+                <!-- <limit effort="15" lower="-1" upper="1.48353" velocity="3.14"/> -->
+                <!-- <dynamics damping="0.7" friction="0.5" /> -->
+                <dynamics damping="10" friction="0" />
             </joint>
             <link name="Right_${prefix}_Phaprox">
@@ -114,5 +120,6 @@
                             rpy="0 0 0" />
                     <mass value="0.0232" />
-                    <inertia ixx="2.5326e-6" ixy="9.2551e-7" ixz="4.0954e-8" iyy="6.9625e-6" iyz="0.0" izz="7.9108e-6" />
+                    <inertia ixx="2.5326e-6" ixy="-9.2551e-7" ixz="-4.0954e-8" iyy="6.9625e-6" iyz="-9.38e-9" izz="7.9108e-6" />
+                    <!-- <inertia ixx="2.5326e-6" ixy="0" ixz="0" iyy="2.9625e-6" iyz="0" izz="2.9108e-6" /> -->
                 </inertial>
                 <visual>
@@ -149,6 +156,8 @@
                 <child link="Right_${prefix}_Phamed" />
                 <axis xyz="0 0 1" />
-                <limit effort="15" lower="0" upper="1.13446" velocity="3.14"/>
-                <dynamics damping="0.7" friction="0.5" />
+                <limit effort="15" lower="0.0872665" upper="1.13446" velocity="3.14"/>
+                <!-- <limit effort="15" lower="-1" upper="1.13446" velocity="3.14"/> -->
+                <!-- <dynamics damping="0.7" friction="0.5" /> -->
+                <dynamics damping="10" friction="0" />
             </joint>
             <link name="Right_${prefix}_Phamed">
@@ -156,5 +165,6 @@
                     <origin xyz="0.0097 -0.00036 0" rpy="0 0 0" />
                     <mass value="0.0158" />
-                    <inertia ixx="1.1852e-6" ixy="2.8845e-8" ixz="6.1323e-9" iyy="2.4460e-6" iyz="2.4541e-9" izz="2.6537e-6" />
+                    <inertia ixx="1.1852e-6" ixy="-2.8845e-8" ixz="-6.1323e-9" iyy="2.4460e-6" iyz="2.4541e-9" izz="2.6537e-6" />
+                    <!-- <inertia ixx="1.1852e-6" ixy="0" ixz="0" iyy="2.4460e-6" iyz="0" izz="2.6537e-6" /> -->
                 </inertial>
                 <visual>
@@ -191,6 +201,7 @@
                 <axis xyz="0 0 1" />
                 <!-- <limit effort="15" lower="-1" upper="1" velocity="3.14"/> -->
-                <limit effort="15" lower="-0.50" upper="1.4" velocity="3.14"/>
-                <dynamics damping="0.7" friction="0.5" />
+                <limit effort="15" lower="0.0872665" upper="1.13446" velocity="3.14"/>
+                <!-- <dynamics damping="0.7" friction="0.5" /> -->
+                <dynamics damping="10" friction="0" />
             </joint>
             <link name="Right_${prefix}_Phadist">
@@ -198,5 +209,6 @@
                     <origin xyz="0.00072 0.00717 0.0" rpy="0 0 0" />
                     <mass value="0.0137" />
-                    <inertia ixx="1.5519e-6" ixy="0.0" ixz="0.0" iyy="8.2972e-7" iyz="0.0" izz="1.5788e-6" />
+                    <inertia ixx="1.5519e-6" ixy="-2.037e-9" ixz="0.0" iyy="8.2972e-7" iyz="3.77e-9" izz="1.5788e-6" />
+                    <!-- <inertia ixx="1.5519e-6" ixy="0" ixz="0" iyy="1.2972e-6" iyz="0" izz="1.5788e-6" /> -->
                 </inertial>
                 <visual>
