Commit message: perf: turn gravity off and set friction in .gazebo file

File: hithand_description/urdf/hithand.xacro (robot description, xacro)
@@ -49,12 +49,4 @@
         		    <mesh filename="package://hithand_description/meshes/collision/hit-hand-2-palm-right.dae"/>
       		    </geometry>
-                <surface>
-                    <friction>
-                        <ode>
-                            <mu>0.8</mu>
-                            <mu2>0.8</mu2>
-                        </ode>
-                    </friction>
-                </surface>
     	    </collision>
         </link>
@@ -79,6 +71,5 @@
                 <axis xyz="0 0 1" />
                 <limit effort="15" lower="-0.261799" upper="0.261799" velocity="3.14"/>
-                <!-- <dynamics damping="0.7" friction="0.5" /> -->
-                <dynamics damping="10" friction="0" />
+                <dynamics damping="0.5" friction="0" />
             </joint>
             <link name="Right_${prefix}_Basecover">
@@ -110,8 +101,6 @@
                 <child link="Right_${prefix}_Phaprox" />
                 <axis xyz="0 0 1" />
-                <limit effort="15" lower="0.0872665" upper="1.48353" velocity="3.14"/>
-                <!-- <limit effort="15" lower="-1" upper="1.48353" velocity="3.14"/> -->
-                <!-- <dynamics damping="0.7" friction="0.5" /> -->
-                <dynamics damping="10" friction="0" />
+                <limit effort="1.15" lower="0.0872665" upper="1.48353" velocity="3.14"/> <!-- Effort limit based on max fingertip force of 10N. Finger tip is approx 11.5cm away from this joint.-->
+                <dynamics damping="0.5" friction="0" />
             </joint>
             <link name="Right_${prefix}_Phaprox">
@@ -140,12 +129,4 @@
                                 <mesh filename="package://hithand_description/meshes/collision/finger/hit-hand-2-finger-phaprox.dae" />
                         </geometry>
-                    <surface>
-                        <friction>
-                            <ode>
-                                <mu>0.8</mu>
-                                <mu2>0.8</mu2>
-                            </ode>
-                        </friction>
-                    </surface>
                 </collision>
             </link>
@@ -156,8 +137,6 @@
                 <child link="Right_${prefix}_Phamed" />
                 <axis xyz="0 0 1" />
-                <limit effort="15" lower="0.0872665" upper="1.13446" velocity="3.14"/>
-                <!-- <limit effort="15" lower="-1" upper="1.13446" velocity="3.14"/> -->
-                <!-- <dynamics damping="0.7" friction="0.5" /> -->
-                <dynamics damping="10" friction="0" />
+                <limit effort="0.6" lower="0.0872665" upper="1.13446" velocity="3.14"/> <!-- Effort limit based on max fingertip force of 10N. Finger tip is approx 6cm away from this joint.-->
+                <dynamics damping="0.5" friction="0" />
             </joint>
             <link name="Right_${prefix}_Phamed">
@@ -184,12 +163,4 @@
                                 <mesh filename="package://hithand_description/meshes/collision/finger/hit-hand-2-finger-phamed.dae" />
                         </geometry>
-                    <surface>
-                        <friction>
-                            <ode>
-                                <mu>0.6</mu>
-                                <mu2>0.6</mu2>
-                            </ode>
-                        </friction>
-                    </surface>
                 </collision>
             </link>
@@ -200,8 +171,6 @@
                 <child link="Right_${prefix}_Phadist" />
                 <axis xyz="0 0 1" />
-                <!-- <limit effort="15" lower="-1" upper="1" velocity="3.14"/> -->
-                <limit effort="15" lower="0.0872665" upper="1.13446" velocity="3.14"/>
-                <!-- <dynamics damping="0.7" friction="0.5" /> -->
-                <dynamics damping="10" friction="0" />
+                <limit effort="0.35" lower="0.0872665" upper="1.13446" velocity="3.14"/> <!-- Effort limit based on max fingertip force of 10N. Finger tip is approx 3.5cm away from this joint.-->
+                <dynamics damping="0.5" friction="0" />
             </joint>
             <link name="Right_${prefix}_Phadist">
@@ -228,12 +197,4 @@
                                 <mesh filename="package://hithand_description/meshes/collision/finger/hit-hand-2-finger-phadist.dae" />
                         </geometry>
-                    <surface>
-                        <friction>
-                            <ode>
-                                <mu>0.8</mu>
-                                <mu2>0.8</mu2>
-                            </ode>
-                        </friction>
-                    </surface>
                 </collision>
             </link>

Commit message: perf: use improved mesh by default

File: hithand_description/urdf/hithand.xacro (robot description, xacro)
@@ -47,5 +47,5 @@
                 <origin rpy="0 0 0" xyz="0 0 0" />
       		    <geometry>
-        		    <mesh filename="package://hithand_description/meshes/collision/hit-hand-2-palm-right.dae"/>
+        		    <mesh filename="package://hithand_description/meshes/collision/hit-hand-2-palm-right-merged.dae"/>
       		    </geometry>
     	    </collision>

Commit message: perf: slightly change position of hithand palm link

File: hithand_description/urdf/hithand.xacro (robot description, xacro)
@@ -56,5 +56,5 @@
             <parent link="base_link_hithand"/>
             <child link="palm_link_hithand"/>
-            <origin xyz="0.02 0 0.06" rpy="-0.15 -1.15 0"/>
+            <origin xyz="0.02 0 0.06" rpy="-0.15 -1.3 0"/>
         </joint>
         <link name="palm_link_hithand"/>

Commit message: perf: increase the base joint range

File: hithand_description/urdf/hithand.xacro (robot description, xacro)
@@ -4,8 +4,4 @@
         <xacro:property name="mu1" value="0.6"/>
         <xacro:property name="mu2" value="0.6"/>
-        <xacro:property name="inertia_mag_0" value="6"/> <!-- should be 5 -->
-        <xacro:property name="inertia_mag_1" value="6"/> <!-- should be 5 -->
-        <xacro:property name="inertia_mag_2" value="6"/> <!-- should be 6 -->
-        <xacro:property name="inertia_mag_3" value="6"/> <!-- should be 6 -->
         <!-- Either attach the Hithand to the then here defined world link or attach to given robot link which itself defines the world frame -->
         <xacro:if value="${not attached}">
@@ -61,5 +57,6 @@
         <!-- #########################FINGER######################## -->
         <!-- Define the fingers in a macro (all fingers are equal) -->
-        <!-- Joint limits set according to this: https://github.com/Qianboy/hithand_ros/blob/master/hithand_description/parameter.pdf -->
+        <!-- Joint limits set according to this: https://github.com/Qianboy/hithand_ros/blob/master/hithand_description/parameter.pdf
+        Note: Following a discussion with Qian Feng, joint limits will be set from 0.0872665 rad to 0.0 rad-->
         <xacro:macro name="finger" params="prefix *transform_palm2finger">
             <!-- +++++ Finger base joint 0 ++++++ -->
@@ -101,5 +98,5 @@
                 <child link="Right_${prefix}_Phaprox" />
                 <axis xyz="0 0 1" />
-                <limit effort="1.15" lower="0.0872665" upper="1.48353" velocity="3.14"/> <!-- Effort limit based on max fingertip force of 10N. Finger tip is approx 11.5cm away from this joint.-->
+                <limit effort="1.15" lower="0.0" upper="1.48353" velocity="3.14"/> <!-- Effort limit based on max fingertip force of 10N. Finger tip is approx 11.5cm away from this joint.-->
                 <dynamics damping="0.5" friction="0" />
             </joint>
@@ -137,5 +134,5 @@
                 <child link="Right_${prefix}_Phamed" />
                 <axis xyz="0 0 1" />
-                <limit effort="0.6" lower="0.0872665" upper="1.13446" velocity="3.14"/> <!-- Effort limit based on max fingertip force of 10N. Finger tip is approx 6cm away from this joint.-->
+                <limit effort="0.6" lower="0.0" upper="1.13446" velocity="3.14"/> <!-- Effort limit based on max fingertip force of 10N. Finger tip is approx 6cm away from this joint.-->
                 <dynamics damping="0.5" friction="0" />
             </joint>
@@ -171,5 +168,5 @@
                 <child link="Right_${prefix}_Phadist" />
                 <axis xyz="0 0 1" />
-                <limit effort="0.35" lower="0.0872665" upper="1.13446" velocity="3.14"/> <!-- Effort limit based on max fingertip force of 10N. Finger tip is approx 3.5cm away from this joint.-->
+                <limit effort="0.35" lower="0.0" upper="1.13446" velocity="3.14"/> <!-- Effort limit based on max fingertip force of 10N. Finger tip is approx 3.5cm away from this joint.-->
                 <dynamics damping="0.5" friction="0" />
             </joint>

Commit message: chore: remove unneccesary comments

File: hithand_description/urdf/hithand.xacro (robot description, xacro)
@@ -27,5 +27,4 @@
       		    <mass value="1.1485"/>
       		    <inertia ixx="2.2458e-3" ixy="-2.7421e-4" ixz="1.6e-5" iyy="2.2203e-3" iyz="-6.37e-5" izz="1.9003e-3" />
-                <!-- <inertia ixx="2.2458e-4" ixy="0" ixz="0" iyy="2.2203e-4" iyz="0" izz="1.9003e-4" /> -->
     	    </inertial>
    	        <visual>
@@ -37,8 +36,4 @@
     	    </visual>
     	    <collision>
-      		    <!-- <origin rpy="0 0 0" xyz="0 0 0.05" />
-      		    <geometry name="hithand_right_palm_collision">
-        		    <box size="0.06 0.1 0.07" />
-      		    </geometry> -->
                 <origin rpy="0 0 0" xyz="0 0 0" />
       		    <geometry>
@@ -48,5 +43,5 @@
         </link>
         <!-- Add a virtual palm link to get the transform of this point via TF for grasping (we align this frame with
-        a normal of an object point cloud.) -->
+        a normal of a point from an object point cloud.) -->
         <joint name="hithand_palm_joint" type="fixed">
             <parent link="base_link_hithand"/>
@@ -58,5 +53,5 @@
         <!-- Define the fingers in a macro (all fingers are equal) -->
         <!-- Joint limits set according to this: https://github.com/Qianboy/hithand_ros/blob/master/hithand_description/parameter.pdf
-        Note: Following a discussion with Qian Feng, joint limits will be set from 0.0872665 rad to 0.0 rad-->
+        Note: Following a discussion with Qian Feng, joint limits will be set from 0.0872665 (msoftware limit) rad to 0.0 (mechanical limit) rad-->
         <xacro:macro name="finger" params="prefix *transform_palm2finger">
             <!-- +++++ Finger base joint 0 ++++++ -->
@@ -73,8 +68,6 @@
                 <inertial>
                     <origin xyz="0.02749 0 0" rpy="0 0 0" />
-                    <!-- <mass value="0.0176" /> -->
                     <mass value="0.0176"/>
                     <inertia ixx="1.3450e-6" ixy="0.0" ixz="-1.8183e-7" iyy="1.9874e-6" iyz="0.0" izz="1.0419e-6" />
-                    <!-- <inertia ixx="1.3450e-6" ixy="0.0" ixz="0" iyy="1.9874e-6" iyz="0.0" izz="1.0419e-6" /> -->
                 </inertial>
                 <visual>
@@ -107,5 +100,4 @@
                     <mass value="0.0232" />
                     <inertia ixx="2.5326e-6" ixy="-9.2551e-7" ixz="-4.0954e-8" iyy="6.9625e-6" iyz="-9.38e-9" izz="7.9108e-6" />
-                    <!-- <inertia ixx="2.5326e-6" ixy="0" ixz="0" iyy="2.9625e-6" iyz="0" izz="2.9108e-6" /> -->
                 </inertial>
                 <visual>
@@ -117,9 +109,4 @@
                 </visual>
                 <collision>
-                    <!-- <origin xyz="0.03 0 0"
-                            rpy="0 0 0" />
-                    <geometry name='hithand_${prefix}_phaprox'>
-                        <box size="0.03 0.03 0.02" />
-                    </geometry> -->
                     <origin xyz="0 0 0" rpy="0 0 0" />
                         <geometry>
@@ -142,5 +129,4 @@
                     <mass value="0.0158" />
                     <inertia ixx="1.1852e-6" ixy="-2.8845e-8" ixz="-6.1323e-9" iyy="2.4460e-6" iyz="2.4541e-9" izz="2.6537e-6" />
-                    <!-- <inertia ixx="1.1852e-6" ixy="0" ixz="0" iyy="2.4460e-6" iyz="0" izz="2.6537e-6" /> -->
                 </inertial>
                 <visual>
@@ -152,8 +138,4 @@
                 </visual>
                 <collision>
-                    <!-- <origin xyz="0.01 0 0" rpy="0 0 0" />
-                    <geometry name='hithand_${prefix}_phamed'>
-                        <box size="0.01 0.02 0.02" />
-                    </geometry> -->
                     <origin xyz="0 0 0" rpy="0 0 0" />
                         <geometry>
@@ -176,5 +158,4 @@
                     <mass value="0.0137" />
                     <inertia ixx="1.5519e-6" ixy="-2.037e-9" ixz="0.0" iyy="8.2972e-7" iyz="3.77e-9" izz="1.5788e-6" />
-                    <!-- <inertia ixx="1.5519e-6" ixy="0" ixz="0" iyy="1.2972e-6" iyz="0" izz="1.5788e-6" /> -->
                 </inertial>
                 <visual>
@@ -186,8 +167,4 @@
                 </visual>
                 <collision>
-                    <!-- <origin xyz="0 0.01 0" rpy="0 0 0" />
-                    <geometry name='hithand_${prefix}_phadist'>
-                        <box size="0.02 0.035 0.02" />
-                    </geometry> -->
                     <origin xyz="0 0 0" rpy="0 0 0" />
                         <geometry>

Commit message: feat: filled all holes of the hand visual models, blender files for this are in blender folder. Exporting to dae did not work, to obj did work. Manually set all Ambient settings to 0.3/0.4 otherwise models would be white. There are now "weird" shadows in the models but no holes

File: hithand_description/urdf/hithand.xacro (robot description, xacro)
@@ -31,5 +31,5 @@
       		    <origin rpy="0 0 0" xyz="0 0 0" />
       		    <geometry>
-        		    <mesh filename="package://hithand_description/meshes/visual/palm/hit-hand-2-palm-right.dae"/>
+        		    <mesh filename="package://hithand_description/meshes/visual/palm/hit-hand-2-palm-right.obj"/>
       		    </geometry>
       		    <material name="grey" />
@@ -104,5 +104,5 @@
                     <origin xyz="0 0 0" rpy="0 0 0" />
                         <geometry>
-                                <mesh filename="package://hithand_description/meshes/visual/finger/hit-hand-2-finger-phaprox.dae" />
+                                <mesh filename="package://hithand_description/meshes/visual/finger/hit-hand-2-finger-phaprox.obj" />
                         </geometry>
                     <material name="lightblue"/>
@@ -133,5 +133,5 @@
                     <origin xyz="0 0 0" rpy="0 0 0" />
                     <geometry>
-                        <mesh filename="package://hithand_description/meshes/visual/finger/hit-hand-2-finger-phamed.dae" />
+                        <mesh filename="package://hithand_description/meshes/visual/finger/hit-hand-2-finger-phamed.obj" />
                     </geometry>
                     <material name="white"/>
@@ -162,5 +162,5 @@
                     <origin xyz="0 0 0" rpy="0 0 0" />
                     <geometry>
-                        <mesh filename="package://hithand_description/meshes/visual/finger/hit-hand-2-finger-phadist.dae" />
+                        <mesh filename="package://hithand_description/meshes/visual/finger/hit-hand-2-finger-phadist.obj" />
                     </geometry>
                     <material name="lightblue"/>

Commit message: add modified version

File: hithand_description/urdf/hithand.xacro (robot description, xacro)
@@ -4,5 +4,5 @@
         <xacro:property name="mu1" value="0.6"/>
         <xacro:property name="mu2" value="0.6"/>
-        <!-- Either attach the Hithand to the then here defined world link or attach to given robot link which itself defines the world frame -->
+        <!-- Either attach the hithand to the then here defined world link or attach to given robot link which itself defines the world frame -->
         <xacro:if value="${not attached}">
         <link name="world"/>
@@ -31,5 +31,5 @@
       		    <origin rpy="0 0 0" xyz="0 0 0" />
       		    <geometry>
-        		    <mesh filename="package://hithand_description/meshes/visual/palm/hit-hand-2-palm-right.obj"/>
+        		    <mesh filename="package://hithand_description/meshes/visual/palm/ar-hand-2-palm-right.dae"/>
       		    </geometry>
       		    <material name="grey" />
@@ -38,5 +38,5 @@
                 <origin rpy="0 0 0" xyz="0 0 0" />
       		    <geometry>
-        		    <mesh filename="package://hithand_description/meshes/collision/palm/hit-hand-2-palm-right-merged.dae"/>
+        		    <mesh filename="package://hithand_description/meshes/collision/palm/ar-hand-2-palm-right-merged.dae"/>
       		    </geometry>
     	    </collision>
@@ -74,5 +74,5 @@
                     <origin xyz="0 0 0" rpy="0 0 0" />
                     <geometry>
-                        <mesh filename="package://hithand_description/meshes/visual/finger/hit-hand-2-finger-basecover.dae"/>
+                        <mesh filename="package://hithand_description/meshes/visual/finger/ar-hand-2-finger-basecover.dae"/>
                     </geometry>
                     <material name="white"/>
@@ -104,5 +104,5 @@
                     <origin xyz="0 0 0" rpy="0 0 0" />
                         <geometry>
-                                <mesh filename="package://hithand_description/meshes/visual/finger/hit-hand-2-finger-phaprox.obj" />
+                                <mesh filename="package://hithand_description/meshes/visual/finger/ar-hand-2-finger-phaprox.dae" />
                         </geometry>
                     <material name="lightblue"/>
@@ -111,5 +111,5 @@
                     <origin xyz="0 0 0" rpy="0 0 0" />
                         <geometry>
-                                <mesh filename="package://hithand_description/meshes/collision/finger/hit-hand-2-finger-phaprox.dae" />
+                                <mesh filename="package://hithand_description/meshes/collision/finger/ar-hand-2-finger-phaprox.dae" />
                         </geometry>
                 </collision>
@@ -133,5 +133,5 @@
                     <origin xyz="0 0 0" rpy="0 0 0" />
                     <geometry>
-                        <mesh filename="package://hithand_description/meshes/visual/finger/hit-hand-2-finger-phamed.obj" />
+                        <mesh filename="package://hithand_description/meshes/visual/finger/ar-hand-2-finger-phamed.dae" />
                     </geometry>
                     <material name="white"/>
@@ -140,5 +140,5 @@
                     <origin xyz="0 0 0" rpy="0 0 0" />
                         <geometry>
-                                <mesh filename="package://hithand_description/meshes/collision/finger/hit-hand-2-finger-phamed.dae" />
+                                <mesh filename="package://hithand_description/meshes/collision/finger/ar-hand-2-finger-phamed.dae" />
                         </geometry>
                 </collision>
@@ -162,5 +162,5 @@
                     <origin xyz="0 0 0" rpy="0 0 0" />
                     <geometry>
-                        <mesh filename="package://hithand_description/meshes/visual/finger/hit-hand-2-finger-phadist.obj" />
+                        <mesh filename="package://hithand_description/meshes/visual/finger/ar-hand-2-finger-phadist.dae" />
                     </geometry>
                     <material name="lightblue"/>
@@ -169,5 +169,5 @@
                     <origin xyz="0 0 0" rpy="0 0 0" />
                         <geometry>
-                                <mesh filename="package://hithand_description/meshes/collision/finger/hit-hand-2-finger-phadist.dae" />
+                                <mesh filename="package://hithand_description/meshes/collision/finger/ar-hand-2-finger-phadist.dae" />
                         </geometry>
                 </collision>

Commit message: feat: add collision body obj

File: hithand_description/urdf/hithand.xacro (robot description, xacro)
@@ -38,5 +38,5 @@
                 <origin rpy="0 0 0" xyz="0 0 0" />
       		    <geometry>
-        		    <mesh filename="package://hithand_description/meshes/collision/palm/hit-hand-2-palm-right-merged.dae"/>
+        		    <mesh filename="package://hithand_description/meshes/collision/palm/hit-hand-2-palm-right-merged.obj"/>
       		    </geometry>
     	    </collision>
@@ -111,5 +111,5 @@
                     <origin xyz="0 0 0" rpy="0 0 0" />
                         <geometry>
-                                <mesh filename="package://hithand_description/meshes/collision/finger/hit-hand-2-finger-phaprox.dae" />
+                                <mesh filename="package://hithand_description/meshes/collision/finger/hit-hand-2-finger-phaprox.obj" />
                         </geometry>
                 </collision>
@@ -140,5 +140,5 @@
                     <origin xyz="0 0 0" rpy="0 0 0" />
                         <geometry>
-                                <mesh filename="package://hithand_description/meshes/collision/finger/hit-hand-2-finger-phamed.dae" />
+                                <mesh filename="package://hithand_description/meshes/collision/finger/hit-hand-2-finger-phamed.obj" />
                         </geometry>
                 </collision>
@@ -169,5 +169,5 @@
                     <origin xyz="0 0 0" rpy="0 0 0" />
                         <geometry>
-                                <mesh filename="package://hithand_description/meshes/collision/finger/hit-hand-2-finger-phadist.dae" />
+                                <mesh filename="package://hithand_description/meshes/collision/finger/hit-hand-2-finger-phadist.obj" />
                         </geometry>
                 </collision>
