Commit message: add gazebo tags to hithand urdf file

File: hithand_description/urdf/hithand.urdf (robot description, URDF)
Before this commit: robot hithand, 22 links, 21 joints
Links:
- link Right_Index_Basecover: geometry collision cylinder length=0.001 radius=0.001; visual mesh filename=package://hithand_description/meshes/visual/hit-hand-2-fing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
- link Right_Index_Phadist: geometry collision mesh filename=package://hithand_description/meshes/visual/hit-hand-2-fing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; visual mesh filename=package://hithand_description/meshes/visual/hit-hand-2-fing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
- link Right_Index_Phamed: geometry collision box size=0.01 0.02 0.02; visual mesh filename=package://hithand_description/meshes/visual/hit-hand-2-fing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
- link Right_Index_Phoaprox: geometry collision box size=0.03 0.03 0.02; visual mesh filename=package://hithand_description/meshes/visual/hit-hand-2-fing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
- link Right_Little_Basecover: geometry collision cylinder length=0.001 radius=0.001; visual mesh filename=package://hithand_description/meshes/visual/hit-hand-2-fing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
- link Right_Little_Phadist: geometry collision mesh filename=package://hithand_description/meshes/visual/hit-hand-2-fing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; visual mesh filename=package://hithand_description/meshes/visual/hit-hand-2-fing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
- link Right_Little_Phamed: geometry collision box size=0.01 0.02 0.02; visual mesh filename=package://hithand_description/meshes/visual/hit-hand-2-fing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
- link Right_Little_Phoaprox: geometry collision box size=0.03 0.03 0.02; visual mesh filename=package://hithand_description/meshes/visual/hit-hand-2-fing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
- link Right_Middle_Basecover: geometry collision cylinder length=0.001 radius=0.001; visual mesh filename=package://hithand_description/meshes/visual/hit-hand-2-fing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
- link Right_Middle_Phadist: geometry collision mesh filename=package://hithand_description/meshes/visual/hit-hand-2-fing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; visual mesh filename=package://hithand_description/meshes/visual/hit-hand-2-fing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
- link Right_Middle_Phamed: geometry collision box size=0.01 0.02 0.02; visual mesh filename=package://hithand_description/meshes/visual/hit-hand-2-fing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
- link Right_Middle_Phoaprox: geometry collision box size=0.03 0.03 0.02; visual mesh filename=package://hithand_description/meshes/visual/hit-hand-2-fing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
- link Right_Ring_Basecover: geometry collision cylinder length=0.001 radius=0.001; visual mesh filename=package://hithand_description/meshes/visual/hit-hand-2-fing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
- link Right_Ring_Phadist: geometry collision mesh filename=package://hithand_description/meshes/visual/hit-hand-2-fing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; visual mesh filename=package://hithand_description/meshes/visual/hit-hand-2-fing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
- link Right_Ring_Phamed: geometry collision box size=0.01 0.02 0.02; visual mesh filename=package://hithand_description/meshes/visual/hit-hand-2-fing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
- link Right_Ring_Phoaprox: geometry collision box size=0.03 0.03 0.02; visual mesh filename=package://hithand_description/meshes/visual/hit-hand-2-fing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
- link Right_Thumb_Basecover: geometry collision cylinder length=0.001 radius=0.001; visual mesh filename=package://hithand_description/meshes/visual/hit-hand-2-fing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
- link Right_Thumb_Phadist: geometry collision mesh filename=package://hithand_description/meshes/visual/hit-hand-2-fing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; visual mesh filename=package://hithand_description/meshes/visual/hit-hand-2-fing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
- link Right_Thumb_Phamed: geometry collision box size=0.01 0.02 0.02; visual mesh filename=package://hithand_description/meshes/visual/hit-hand-2-fing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
- link Right_Thumb_Phoaprox: geometry collision box size=0.03 0.03 0.02; visual mesh filename=package://hithand_description/meshes/visual/hit-hand-2-fing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
- link base_link: geometry collision mesh filename=package://hithand_description/meshes/visual/hit-hand-2-palm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; visual mesh filename=package://hithand_description/meshes/visual/hit-hand-2-palm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

Commit message: One finger version of hithand to be tested of ros control

File: hithand_description/urdf/hithand.urdf (robot description, URDF)
Before this commit: robot hithand, 22 links, 21 joints
Links:
- removed link Right_Index_Basecover
- removed link Right_Index_Phadist
- removed link Right_Index_Phamed
- removed link Right_Index_Phoaprox
- removed link Right_Little_Basecover
- removed link Right_Little_Phadist
- removed link Right_Little_Phamed
- removed link Right_Little_Phoaprox
- removed link Right_Middle_Basecover
- removed link Right_Middle_Phadist
- removed link Right_Middle_Phamed
- removed link Right_Middle_Phoaprox
- removed link Right_Ring_Basecover
- removed link Right_Ring_Phadist
- removed link Right_Ring_Phamed
- removed link Right_Ring_Phoaprox
Joints:
- removed joint Right_Index_1
- removed joint Right_Index_2
- removed joint Right_Index_3
- removed joint Right_Index_4
- removed joint Right_Little_1
- removed joint Right_Little_2
- removed joint Right_Little_3
- removed joint Right_Little_4
- removed joint Right_Middle_1
- removed joint Right_Middle_2
- removed joint Right_Middle_3
- removed joint Right_Middle_4
- removed joint Right_Ring_1
- removed joint Right_Ring_2
- removed joint Right_Ring_3
- removed joint Right_Ring_4
- joint Right_Thumb_1: limit lower=-0.50 upper=1.4 effort=30 velocity=3.14 -> lower=-0.50 upper=1.4 effort=1000 velocity=3.14
- joint Right_Thumb_2: limit lower=-0.50 upper=1.4 effort=30 velocity=3.14 -> lower=-0.50 upper=1.4 effort=1000 velocity=3.14
- joint Right_Thumb_3: limit lower=-0.50 upper=1.4 effort=30 velocity=3.14 -> lower=-0.50 upper=1.4 effort=1000 velocity=3.14
- joint Right_Thumb_4: limit lower=-0.50 upper=1.4 effort=30 velocity=3.14 -> lower=-0.50 upper=1.4 effort=1000 velocity=3.14

File: hithand_description/urdf/hithand.xacro (robot description, xacro)
@@ -72,5 +72,6 @@
             <child link="Right_${prefix}_Basecover" />
         <axis xyz="0 0 1" />
-        <limit effort="30" lower="-0.50" upper="1.4" velocity="3.14"/>
+        <limit effort="1000" lower="-0.50" upper="1.4" velocity="3.14"/>
+          <dynamics damping="0.7" friction="0.5" />
       </joint>
       <link name="Right_${prefix}_Phoaprox">
@@ -112,5 +113,6 @@
             <child link="Right_${prefix}_Phoaprox" />
             <axis xyz="0 0 1" />
-            <limit effort="30" lower="-0.50" upper="1.4" velocity="3.14"/>
+            <limit effort="1000" lower="-0.50" upper="1.4" velocity="3.14"/>
+            <dynamics damping="0.7" friction="0.5" />
       </joint>
       <link name="Right_${prefix}_Phamed">
@@ -152,5 +154,6 @@
             <child link="Right_${prefix}_Phamed" />
             <axis xyz="0 0 1" />
-            <limit effort="30" lower="-0.50" upper="1.4" velocity="3.14"/>
+            <limit effort="1000" lower="-0.50" upper="1.4" velocity="3.14"/>
+          <dynamics damping="0.7" friction="0.5" />
       </joint>
       <link name="Right_${prefix}_Phadist">
@@ -192,5 +195,6 @@
             <child link="Right_${prefix}_Phadist" />
             <axis xyz="0 0 1" />
-            <limit effort="30" lower="-0.50" upper="1.4" velocity="3.14"/>
+            <limit effort="1000" lower="-0.50" upper="1.4" velocity="3.14"/>
+          <dynamics damping="0.7" friction="0.5" />
       </joint>
     </xacro:macro>
@@ -200,19 +204,19 @@
             rpy="0.225810 -1.083656 0.411355" />
     </xacro:finger>
-    <xacro:finger prefix="Index"  >
-        <origin xyz="-0.002529881 0.03680013 0.107783545"
-      		rpy="3.054326 -1.570796 0.000000" />
-    </xacro:finger>
-    <xacro:finger prefix="Middle"  >
-            <origin xyz="-0.0037 0.01  0.117783545"
-      		rpy="-3.141593 -1.570796 0.000000" />
-    </xacro:finger>
-    <xacro:finger prefix="Ring"   >
-            <origin xyz="0 -0.01680013 0.11258354"
-            rpy="-3.054326 -1.570796 0.000000" />
-    </xacro:finger>
-    <xacro:finger prefix="Little"  >
-            <origin xyz="0.000971571 -0.0433963 0.093583545"
-            rpy="-2.967060 -1.570796 0.000000" />
-    </xacro:finger>
+<!--    <xacro:finger prefix="Index"  >-->
+<!--        <origin xyz="-0.002529881 0.03680013 0.107783545"-->
+<!--      		rpy="3.054326 -1.570796 0.000000" />-->
+<!--    </xacro:finger>-->
+<!--    <xacro:finger prefix="Middle"  >-->
+<!--            <origin xyz="-0.0037 0.01  0.117783545"-->
+<!--      		rpy="-3.141593 -1.570796 0.000000" />-->
+<!--    </xacro:finger>-->
+<!--    <xacro:finger prefix="Ring"   >-->
+<!--            <origin xyz="0 -0.01680013 0.11258354"-->
+<!--            rpy="-3.054326 -1.570796 0.000000" />-->
+<!--    </xacro:finger>-->
+<!--    <xacro:finger prefix="Little"  >-->
+<!--            <origin xyz="0.000971571 -0.0433963 0.093583545"-->
+<!--            rpy="-2.967060 -1.570796 0.000000" />-->
+<!--    </xacro:finger>-->
 </robot>

File: hithand_description/urdf/transmission.xacro (robot description, xacro)
@@ -6,8 +6,8 @@
       <type>transmission_interface/SimpleTransmission</type>
       <joint name="Right_${finger_name}_1">
-        <hardwareInterface>EffortJointInterface</hardwareInterface>
+        <hardwareInterface>hardware_interface/PositionJointInterface</hardwareInterface>
       </joint>
       <actuator name="motor_${finger_name}_1">
-        <hardwareInterface>EffortJointInterface</hardwareInterface>
+        <hardwareInterface>hardware_interface/PositionJointInterface</hardwareInterface>
         <mechanicalReduction>1</mechanicalReduction>
       </actuator>
@@ -16,8 +16,8 @@
         <type>transmission_interface/SimpleTransmission</type>
         <joint name="Right_${finger_name}_2">
-          <hardwareInterface>EffortJointInterface</hardwareInterface>
+          <hardwareInterface>hardware_interface/PositionJointInterface</hardwareInterface>
         </joint>
         <actuator name="motor_${finger_name}_2">
-          <hardwareInterface>EffortJointInterface</hardwareInterface>
+          <hardwareInterface>hardware_interface/PositionJointInterface</hardwareInterface>
           <mechanicalReduction>1</mechanicalReduction>
         </actuator>
@@ -26,8 +26,8 @@
         <type>transmission_interface/SimpleTransmission</type>
         <joint name="Right_${finger_name}_3">
-          <hardwareInterface>EffortJointInterface</hardwareInterface>
+          <hardwareInterface>hardware_interface/PositionJointInterface</hardwareInterface>
         </joint>
         <actuator name="motor_${finger_name}_3">
-          <hardwareInterface>EffortJointInterface</hardwareInterface>
+          <hardwareInterface>hardware_interface/PositionJointInterface</hardwareInterface>
           <mechanicalReduction>1</mechanicalReduction>
         </actuator>
@@ -36,8 +36,8 @@
         <type>transmission_interface/SimpleTransmission</type>
         <joint name="Right_${finger_name}_4">
-          <hardwareInterface>EffortJointInterface</hardwareInterface>
+          <hardwareInterface>hardware_interface/PositionJointInterface</hardwareInterface>
         </joint>
         <actuator name="motor_${finger_name}_4">
-          <hardwareInterface>EffortJointInterface</hardwareInterface>
+          <hardwareInterface>hardware_interface/PositionJointInterface</hardwareInterface>
           <mechanicalReduction>1</mechanicalReduction>
         </actuator>
@@ -46,11 +46,11 @@
     <xacro:hithand_transmission finger_name="Thumb">
     </xacro:hithand_transmission>
-    <xacro:hithand_transmission finger_name="Index">
-    </xacro:hithand_transmission>
-    <xacro:hithand_transmission finger_name="Middle">
-    </xacro:hithand_transmission>
-    <xacro:hithand_transmission finger_name="Ring">
-    </xacro:hithand_transmission>
-    <xacro:hithand_transmission finger_name="Little">
-    </xacro:hithand_transmission>
+<!--    <xacro:hithand_transmission finger_name="Index">-->
+<!--    </xacro:hithand_transmission>-->
+<!--    <xacro:hithand_transmission finger_name="Middle">-->
+<!--    </xacro:hithand_transmission>-->
+<!--    <xacro:hithand_transmission finger_name="Ring">-->
+<!--    </xacro:hithand_transmission>-->
+<!--    <xacro:hithand_transmission finger_name="Little">-->
+<!--    </xacro:hithand_transmission>-->
 </robot>
