Commit message: Effor controller works from ros control

File: hithand_description/urdf/hithand.urdf (robot description, URDF)
Before this commit: robot hithand, 6 links, 5 joints
Links:
- added link Right_Index_Basecover, mass 1.0; collision cylinder length=0.001 radius=0.001; visual mesh filename=package://hithand_description/meshes/visual/hit-hand-2-fing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
- added link Right_Index_Phadist, mass 1.0; collision mesh filename=package://hithand_description/meshes/visual/hit-hand-2-fing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; visual mesh filename=package://hithand_description/meshes/visual/hit-hand-2-fing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
- added link Right_Index_Phamed, mass 1.0; collision box size=0.01 0.02 0.02; visual mesh filename=package://hithand_description/meshes/visual/hit-hand-2-fing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
- added link Right_Index_Phoaprox, mass 1.0; collision box size=0.03 0.03 0.02; visual mesh filename=package://hithand_description/meshes/visual/hit-hand-2-fing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
- added link Right_Little_Basecover, mass 1.0; collision cylinder length=0.001 radius=0.001; visual mesh filename=package://hithand_description/meshes/visual/hit-hand-2-fing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
- added link Right_Little_Phadist, mass 1.0; collision mesh filename=package://hithand_description/meshes/visual/hit-hand-2-fing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; visual mesh filename=package://hithand_description/meshes/visual/hit-hand-2-fing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
- added link Right_Little_Phamed, mass 1.0; collision box size=0.01 0.02 0.02; visual mesh filename=package://hithand_description/meshes/visual/hit-hand-2-fing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
- added link Right_Little_Phoaprox, mass 1.0; collision box size=0.03 0.03 0.02; visual mesh filename=package://hithand_description/meshes/visual/hit-hand-2-fing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
- added link Right_Middle_Basecover, mass 1.0; collision cylinder length=0.001 radius=0.001; visual mesh filename=package://hithand_description/meshes/visual/hit-hand-2-fing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
- added link Right_Middle_Phadist, mass 1.0; collision mesh filename=package://hithand_description/meshes/visual/hit-hand-2-fing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; visual mesh filename=package://hithand_description/meshes/visual/hit-hand-2-fing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
- added link Right_Middle_Phamed, mass 1.0; collision box size=0.01 0.02 0.02; visual mesh filename=package://hithand_description/meshes/visual/hit-hand-2-fing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
- added link Right_Middle_Phoaprox, mass 1.0; collision box size=0.03 0.03 0.02; visual mesh filename=package://hithand_description/meshes/visual/hit-hand-2-fing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
- added link Right_Ring_Basecover, mass 1.0; collision cylinder length=0.001 radius=0.001; visual mesh filename=package://hithand_description/meshes/visual/hit-hand-2-fing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
- added link Right_Ring_Phadist, mass 1.0; collision mesh filename=package://hithand_description/meshes/visual/hit-hand-2-fing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; visual mesh filename=package://hithand_description/meshes/visual/hit-hand-2-fing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
- added link Right_Ring_Phamed, mass 1.0; collision box size=0.01 0.02 0.02; visual mesh filename=package://hithand_description/meshes/visual/hit-hand-2-fing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
- added link Right_Ring_Phoaprox, mass 1.0; collision box size=0.03 0.03 0.02; visual mesh filename=package://hithand_description/meshes/visual/hit-hand-2-fing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
Joints:
- added joint Right_Index_1: type revolute, parent base_link, child Right_Index_Basecover, origin xyz=-0.002529881 0.03680013 0.107783545 rpy=3.054326 -1.570796 0.000000, axis 0 0 1, limit lower=-0.50 upper=1.4 effort=1000 velocity=3.14
- added joint Right_Index_2: type revolute, parent Right_Index_Basecover, child Right_Index_Phoaprox, origin xyz=0 0 0  rpy=1.5708 0 0, axis 0 0 1, limit lower=-0.50 upper=1.4 effort=1000 velocity=3.14
- added joint Right_Index_3: type revolute, parent Right_Index_Phoaprox, child Right_Index_Phamed, origin xyz=0.055 0 0 rpy=0 0 0, axis 0 0 1, limit lower=-0.50 upper=1.4 effort=1000 velocity=3.14
- added joint Right_Index_4: type revolute, parent Right_Index_Phamed, child Right_Index_Phadist, origin xyz=0.025 0 0 rpy=0 0 -1.57, axis 0 0 1, limit lower=-0.50 upper=1.4 effort=1000 velocity=3.14
- added joint Right_Little_1: type revolute, parent base_link, child Right_Little_Basecover, origin xyz=0.000971571 -0.0433963 0.093583545 rpy=-2.967060 -1.570796 0.000000, axis 0 0 1, limit lower=-0.50 upper=1.4 effort=1000 velocity=3.14
- added joint Right_Little_2: type revolute, parent Right_Little_Basecover, child Right_Little_Phoaprox, origin xyz=0 0 0  rpy=1.5708 0 0, axis 0 0 1, limit lower=-0.50 upper=1.4 effort=1000 velocity=3.14
- added joint Right_Little_3: type revolute, parent Right_Little_Phoaprox, child Right_Little_Phamed, origin xyz=0.055 0 0 rpy=0 0 0, axis 0 0 1, limit lower=-0.50 upper=1.4 effort=1000 velocity=3.14
- added joint Right_Little_4: type revolute, parent Right_Little_Phamed, child Right_Little_Phadist, origin xyz=0.025 0 0 rpy=0 0 -1.57, axis 0 0 1, limit lower=-0.50 upper=1.4 effort=1000 velocity=3.14
- added joint Right_Middle_1: type revolute, parent base_link, child Right_Middle_Basecover, origin xyz=-0.0037 0.01  0.117783545 rpy=-3.141593 -1.570796 0.000000, axis 0 0 1, limit lower=-0.50 upper=1.4 effort=1000 velocity=3.14
- added joint Right_Middle_2: type revolute, parent Right_Middle_Basecover, child Right_Middle_Phoaprox, origin xyz=0 0 0  rpy=1.5708 0 0, axis 0 0 1, limit lower=-0.50 upper=1.4 effort=1000 velocity=3.14
- added joint Right_Middle_3: type revolute, parent Right_Middle_Phoaprox, child Right_Middle_Phamed, origin xyz=0.055 0 0 rpy=0 0 0, axis 0 0 1, limit lower=-0.50 upper=1.4 effort=1000 velocity=3.14
- added joint Right_Middle_4: type revolute, parent Right_Middle_Phamed, child Right_Middle_Phadist, origin xyz=0.025 0 0 rpy=0 0 -1.57, axis 0 0 1, limit lower=-0.50 upper=1.4 effort=1000 velocity=3.14
- added joint Right_Ring_1: type revolute, parent base_link, child Right_Ring_Basecover, origin xyz=0 -0.01680013 0.11258354 rpy=-3.054326 -1.570796 0.000000, axis 0 0 1, limit lower=-0.50 upper=1.4 effort=1000 velocity=3.14
- added joint Right_Ring_2: type revolute, parent Right_Ring_Basecover, child Right_Ring_Phoaprox, origin xyz=0 0 0  rpy=1.5708 0 0, axis 0 0 1, limit lower=-0.50 upper=1.4 effort=1000 velocity=3.14
- added joint Right_Ring_3: type revolute, parent Right_Ring_Phoaprox, child Right_Ring_Phamed, origin xyz=0.055 0 0 rpy=0 0 0, axis 0 0 1, limit lower=-0.50 upper=1.4 effort=1000 velocity=3.14
- added joint Right_Ring_4: type revolute, parent Right_Ring_Phamed, child Right_Ring_Phadist, origin xyz=0.025 0 0 rpy=0 0 -1.57, axis 0 0 1, limit lower=-0.50 upper=1.4 effort=1000 velocity=3.14

File: hithand_description/urdf/hithand.xacro (robot description, xacro)
@@ -204,19 +204,19 @@
             rpy="0.225810 -1.083656 0.411355" />
     </xacro:finger>
-<!--    <xacro:finger prefix="Index"  >-->
-<!--        <origin xyz="-0.002529881 0.03680013 0.107783545"-->
-<!--      		rpy="3.054326 -1.570796 0.000000" />-->
-<!--    </xacro:finger>-->
-<!--    <xacro:finger prefix="Middle"  >-->
-<!--            <origin xyz="-0.0037 0.01  0.117783545"-->
-<!--      		rpy="-3.141593 -1.570796 0.000000" />-->
-<!--    </xacro:finger>-->
-<!--    <xacro:finger prefix="Ring"   >-->
-<!--            <origin xyz="0 -0.01680013 0.11258354"-->
-<!--            rpy="-3.054326 -1.570796 0.000000" />-->
-<!--    </xacro:finger>-->
-<!--    <xacro:finger prefix="Little"  >-->
-<!--            <origin xyz="0.000971571 -0.0433963 0.093583545"-->
-<!--            rpy="-2.967060 -1.570796 0.000000" />-->
-<!--    </xacro:finger>-->
+    <xacro:finger prefix="Index"  >
+        <origin xyz="-0.002529881 0.03680013 0.107783545"
+      		rpy="3.054326 -1.570796 0.000000" />
+    </xacro:finger>
+    <xacro:finger prefix="Middle"  >
+            <origin xyz="-0.0037 0.01  0.117783545"
+      		rpy="-3.141593 -1.570796 0.000000" />
+    </xacro:finger>
+    <xacro:finger prefix="Ring"   >
+            <origin xyz="0 -0.01680013 0.11258354"
+            rpy="-3.054326 -1.570796 0.000000" />
+    </xacro:finger>
+    <xacro:finger prefix="Little"  >
+            <origin xyz="0.000971571 -0.0433963 0.093583545"
+            rpy="-2.967060 -1.570796 0.000000" />
+    </xacro:finger>
 </robot>

File: hithand_description/urdf/transmission.xacro (robot description, xacro)
@@ -6,8 +6,8 @@
       <type>transmission_interface/SimpleTransmission</type>
       <joint name="Right_${finger_name}_1">
-        <hardwareInterface>hardware_interface/PositionJointInterface</hardwareInterface>
+        <hardwareInterface>hardware_interface/EffortJointInterface</hardwareInterface>
       </joint>
       <actuator name="motor_${finger_name}_1">
-        <hardwareInterface>hardware_interface/PositionJointInterface</hardwareInterface>
+        <hardwareInterface>hardware_interface/EffortJointInterface</hardwareInterface>
         <mechanicalReduction>1</mechanicalReduction>
       </actuator>
@@ -16,8 +16,8 @@
         <type>transmission_interface/SimpleTransmission</type>
         <joint name="Right_${finger_name}_2">
-          <hardwareInterface>hardware_interface/PositionJointInterface</hardwareInterface>
+          <hardwareInterface>hardware_interface/EffortJointInterface</hardwareInterface>
         </joint>
         <actuator name="motor_${finger_name}_2">
-          <hardwareInterface>hardware_interface/PositionJointInterface</hardwareInterface>
+          <hardwareInterface>hardware_interface/EffortJointInterface</hardwareInterface>
           <mechanicalReduction>1</mechanicalReduction>
         </actuator>
@@ -26,8 +26,8 @@
         <type>transmission_interface/SimpleTransmission</type>
         <joint name="Right_${finger_name}_3">
-          <hardwareInterface>hardware_interface/PositionJointInterface</hardwareInterface>
+          <hardwareInterface>hardware_interface/EffortJointInterface</hardwareInterface>
         </joint>
         <actuator name="motor_${finger_name}_3">
-          <hardwareInterface>hardware_interface/PositionJointInterface</hardwareInterface>
+          <hardwareInterface>hardware_interface/EffortJointInterface</hardwareInterface>
           <mechanicalReduction>1</mechanicalReduction>
         </actuator>
@@ -36,8 +36,8 @@
         <type>transmission_interface/SimpleTransmission</type>
         <joint name="Right_${finger_name}_4">
-          <hardwareInterface>hardware_interface/PositionJointInterface</hardwareInterface>
+          <hardwareInterface>hardware_interface/EffortJointInterface</hardwareInterface>
         </joint>
         <actuator name="motor_${finger_name}_4">
-          <hardwareInterface>hardware_interface/PositionJointInterface</hardwareInterface>
+          <hardwareInterface>hardware_interface/EffortJointInterface</hardwareInterface>
           <mechanicalReduction>1</mechanicalReduction>
         </actuator>
@@ -46,11 +46,11 @@
     <xacro:hithand_transmission finger_name="Thumb">
     </xacro:hithand_transmission>
-<!--    <xacro:hithand_transmission finger_name="Index">-->
-<!--    </xacro:hithand_transmission>-->
-<!--    <xacro:hithand_transmission finger_name="Middle">-->
-<!--    </xacro:hithand_transmission>-->
-<!--    <xacro:hithand_transmission finger_name="Ring">-->
-<!--    </xacro:hithand_transmission>-->
-<!--    <xacro:hithand_transmission finger_name="Little">-->
-<!--    </xacro:hithand_transmission>-->
+    <xacro:hithand_transmission finger_name="Index">
+    </xacro:hithand_transmission>
+    <xacro:hithand_transmission finger_name="Middle">
+    </xacro:hithand_transmission>
+    <xacro:hithand_transmission finger_name="Ring">
+    </xacro:hithand_transmission>
+    <xacro:hithand_transmission finger_name="Little">
+    </xacro:hithand_transmission>
 </robot>

Commit message: clean up

File: hithand_description/urdf/hithand.urdf (robot description, URDF)
Before this commit: robot hithand, 23 links, 22 joints
Links:
- link base_link_hithand: geometry collision mesh filename=package://hithand_description/meshes/collision/palm/hit-han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; visual mesh filename=package://hithand_description/meshes/visual/palm/hit-hand-2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

File: hithand_description/urdf/hithand.xacro (robot description, xacro)
@@ -36,5 +36,5 @@
       		    <origin rpy="0 0 0" xyz="0 0 0" />
       		    <geometry>
-        		    <mesh filename="package://hithand_description/meshes/visual/hit-hand-2-palm-right.dae"/>
+        		    <mesh filename="package://hithand_description/meshes/visual/palm/hit-hand-2-palm-right.dae"/>
       		    </geometry>
       		    <material name="grey" />
@@ -47,5 +47,5 @@
                 <origin rpy="0 0 0" xyz="0 0 0" />
       		    <geometry>
-        		    <mesh filename="package://hithand_description/meshes/collision/hit-hand-2-palm-right-merged.dae"/>
+        		    <mesh filename="package://hithand_description/meshes/collision/palm/hit-hand-2-palm-right-merged.dae"/>
       		    </geometry>
     	    </collision>

Commit message: feat(hithand.xacro): make world and base_link_hithand identical

File: hithand_description/urdf/hithand.urdf (robot description, URDF)
Before this commit: robot hithand, 23 links, 22 joints
Joints:
- joint fixed: origin xyz=0 0 0.1 rpy=0 0 0 -> xyz=0 0 0 rpy=0 0 0

File: hithand_description/urdf/hithand.xacro (robot description, xacro)
@@ -10,5 +10,5 @@
                 <parent link="world"/>
                 <child link="base_link_hithand"/>
-                <origin xyz="0 0 0.1" rpy="0 0 0"/>
+		<origin xyz="0 0 0" rpy="0 0 0"/>
             </joint>
         </xacro:if>

Commit message: add fingertip virtual frame

File: hithand_description/urdf/hithand.urdf (robot description, URDF)
Before this commit: robot hithand, 23 links, 22 joints
Links:
- added link Right_Index_fingertip
- added link Right_Little_fingertip
- added link Right_Middle_fingertip
- added link Right_Ring_fingertip
- added link Right_Thumb_fingertip
Joints:
- added joint Right_Index_4: type fixed, parent Right_Index_Phadist, child Right_Index_fingertip, origin xyz=0.025 0 0 rpy=0 0 -1.570796
- added joint Right_Little_4: type fixed, parent Right_Little_Phadist, child Right_Little_fingertip, origin xyz=0.025 0 0 rpy=0 0 -1.570796
- added joint Right_Middle_4: type fixed, parent Right_Middle_Phadist, child Right_Middle_fingertip, origin xyz=0.025 0 0 rpy=0 0 -1.570796
- added joint Right_Ring_4: type fixed, parent Right_Ring_Phadist, child Right_Ring_fingertip, origin xyz=0.025 0 0 rpy=0 0 -1.570796
- added joint Right_Thumb_4: type fixed, parent Right_Thumb_Phadist, child Right_Thumb_fingertip, origin xyz=0.025 0 0 rpy=0 0 -1.570796
- joint fixed: origin xyz=0 0 0 rpy=0 0 0 -> xyz=0 0 0.1 rpy=0 0 0

File: hithand_description/urdf/hithand.xacro (robot description, xacro)
@@ -173,4 +173,10 @@
                 </collision>
             </link>
+            <joint name="Right_${prefix}_4" type="fixed">
+                <parent link="Right_${prefix}_Phadist"/>
+                <child link="Right_${prefix}_fingertip"/>
+                <origin xyz="0.025 0 0" rpy="0 0 -1.570796" />
+            </joint>
+            <link name="Right_${prefix}_fingertip"/>
         </xacro:macro>
         <!-- #########################FINGER######################## -->
