Commit message: chore: updated hithand urdf and sdf

File: Models/hithand/hithand.urdf (robot description, URDF)
Before this commit: robot hithand, 22 links, 21 joints
Links:
- removed link Right_Index_Phoaprox
- removed link Right_Little_Phoaprox
- removed link Right_Middle_Phoaprox
- removed link Right_Ring_Phoaprox
- removed link Right_Thumb_Phoaprox
- removed link base_link
- added link Right_Index_Phaprox, mass 0.0232; collision mesh filename=package://hithand_description/meshes/collision/finger/hit-h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; visual mesh filename=package://hithand_description/meshes/visual/finger/hit-hand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
- added link Right_Little_Phaprox, mass 0.0232; collision mesh filename=package://hithand_description/meshes/collision/finger/hit-h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; visual mesh filename=package://hithand_description/meshes/visual/finger/hit-hand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
- added link Right_Middle_Phaprox, mass 0.0232; collision mesh filename=package://hithand_description/meshes/collision/finger/hit-h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; visual mesh filename=package://hithand_description/meshes/visual/finger/hit-hand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
- added link Right_Ring_Phaprox, mass 0.0232; collision mesh filename=package://hithand_description/meshes/collision/finger/hit-h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; visual mesh filename=package://hithand_description/meshes/visual/finger/hit-hand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
- added link Right_Thumb_Phaprox, mass 0.0232; collision mesh filename=package://hithand_description/meshes/collision/finger/hit-h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; visual mesh filename=package://hithand_description/meshes/visual/finger/hit-hand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
- added link base_link_hithand, mass 1.1485; collision mesh filename=package://hithand_description/meshes/collision/palm/hit-han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; visual mesh filename=package://hithand_description/meshes/visual/palm/hit-hand-2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
- added link palm_link_hithand
- link Right_Index_Basecover: mass 1.0 -> 0.0176; geometry collision cylinder length=0.001 radius=0.001; visual mesh filename=package://hithand_description/meshes/visual/finger/hit-hand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
- link Right_Index_Phadist: mass 1.0 -> 0.0137; geometry collision mesh filename=package://hithand_description/meshes/collision/finger/hit-h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; visual mesh filename=package://hithand_description/meshes/visual/finger/hit-hand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
- link Right_Index_Phamed: mass 1.0 -> 0.0158; geometry collision mesh filename=package://hithand_description/meshes/collision/finger/hit-h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; visual mesh filename=package://hithand_description/meshes/visual/finger/hit-hand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
- link Right_Little_Basecover: mass 1.0 -> 0.0176; geometry collision cylinder length=0.001 radius=0.001; visual mesh filename=package://hithand_description/meshes/visual/finger/hit-hand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
- link Right_Little_Phadist: mass 1.0 -> 0.0137; geometry collision mesh filename=package://hithand_description/meshes/collision/finger/hit-h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; visual mesh filename=package://hithand_description/meshes/visual/finger/hit-hand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
- link Right_Little_Phamed: mass 1.0 -> 0.0158; geometry collision mesh filename=package://hithand_description/meshes/collision/finger/hit-h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; visual mesh filename=package://hithand_description/meshes/visual/finger/hit-hand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
- link Right_Middle_Basecover: mass 1.0 -> 0.0176; geometry collision cylinder length=0.001 radius=0.001; visual mesh filename=package://hithand_description/meshes/visual/finger/hit-hand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
- link Right_Middle_Phadist: mass 1.0 -> 0.0137; geometry collision mesh filename=package://hithand_description/meshes/collision/finger/hit-h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; visual mesh filename=package://hithand_description/meshes/visual/finger/hit-hand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
- link Right_Middle_Phamed: mass 1.0 -> 0.0158; geometry collision mesh filename=package://hithand_description/meshes/collision/finger/hit-h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; visual mesh filename=package://hithand_description/meshes/visual/finger/hit-hand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
- link Right_Ring_Basecover: mass 1.0 -> 0.0176; geometry collision cylinder length=0.001 radius=0.001; visual mesh filename=package://hithand_description/meshes/visual/finger/hit-hand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
- link Right_Ring_Phadist: mass 1.0 -> 0.0137; geometry collision mesh filename=package://hithand_description/meshes/collision/finger/hit-h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; visual mesh filename=package://hithand_description/meshes/visual/finger/hit-hand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
- link Right_Ring_Phamed: mass 1.0 -> 0.0158; geometry collision mesh filename=package://hithand_description/meshes/collision/finger/hit-h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; visual mesh filename=package://hithand_description/meshes/visual/finger/hit-hand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
- link Right_Thumb_Basecover: mass 1.0 -> 0.0176; geometry collision cylinder length=0.001 radius=0.001; visual mesh filename=package://hithand_description/meshes/visual/finger/hit-hand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
- link Right_Thumb_Phadist: mass 1.0 -> 0.0137; geometry collision mesh filename=package://hithand_description/meshes/collision/finger/hit-h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; visual mesh filename=package://hithand_description/meshes/visual/finger/hit-hand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
- link Right_Thumb_Phamed: mass 1.0 -> 0.0158; geometry collision mesh filename=package://hithand_description/meshes/collision/finger/hit-h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; visual mesh filename=package://hithand_description/meshes/visual/finger/hit-hand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
Joints:
- removed joint Right_Index_4
- removed joint Right_Little_4
- removed joint Right_Middle_4
- removed joint Right_Ring_4
- removed joint Right_Thumb_4
- added joint Right_Index_0: type revolute, parent base_link_hithand, child Right_Index_Basecover, origin xyz=-0.002529881 0.03680013 0.107783545 rpy=3.054326 -1.570796 0.000000, axis 0 0 1, limit lower=-0.261799 upper=0.261799 effort=15 velocity=3.14
- added joint Right_Little_0: type revolute, parent base_link_hithand, child Right_Little_Basecover, origin xyz=0.000971571 -0.0433963 0.093583545 rpy=-2.967060 -1.570796 0.000000, axis 0 0 1, limit lower=-0.261799 upper=0.261799 effort=15 velocity=3.14
- added joint Right_Middle_0: type revolute, parent base_link_hithand, child Right_Middle_Basecover, origin xyz=-0.0037 0.01  0.117783545 rpy=-3.141593 -1.570796 0.000000, axis 0 0 1, limit lower=-0.261799 upper=0.261799 effort=15 velocity=3.14
- added joint Right_Ring_0: type revolute, parent base_link_hithand, child Right_Ring_Basecover, origin xyz=0 -0.01680013 0.11258354 rpy=-3.054326 -1.570796 0.000000, axis 0 0 1, limit lower=-0.261799 upper=0.261799 effort=15 velocity=3.14
- added joint Right_Thumb_0: type revolute, parent base_link_hithand, child Right_Thumb_Basecover, origin xyz=0.06217593 0.044372912 0.078734808 rpy=0.225810 -1.083656 0.411355, axis 0 0 1, limit lower=-0.261799 upper=0.261799 effort=15 velocity=3.14
- added joint hithand_palm_joint: type fixed, parent base_link_hithand, child palm_link_hithand, origin xyz=0.02 0 0.06 rpy=-0.15 -1.3 0
- joint Right_Index_1: child Right_Index_Basecover -> Right_Index_Phaprox; limit lower=-0.50 upper=1.4 effort=1000 velocity=3.14 -> lower=0.0872665 upper=1.48353 effort=1.15 velocity=3.14; origin xyz=-0.002529881 0.03680013 0.107783545 rpy=3.054326 -1.570796 0.000000 -> xyz=0 0 0  rpy=1.5708 0 0; parent base_link -> Right_Index_Basecover
- joint Right_Index_2: child Right_Index_Phoaprox -> Right_Index_Phamed; limit lower=-0.50 upper=1.4 effort=1000 velocity=3.14 -> lower=0.0872665 upper=1.13446 effort=0.6 velocity=3.14; origin xyz=0 0 0  rpy=1.5708 0 0 -> xyz=0.055 0 0 rpy=0 0 0; parent Right_Index_Basecover -> Right_Index_Phaprox
- joint Right_Index_3: child Right_Index_Phamed -> Right_Index_Phadist; limit lower=-0.50 upper=1.4 effort=1000 velocity=3.14 -> lower=0.0872665 upper=1.13446 effort=0.35 velocity=3.14; origin xyz=0.055 0 0 rpy=0 0 0 -> xyz=0.025 0 0 rpy=0 0 -1.570796; parent Right_Index_Phoaprox -> Right_Index_Phamed
- joint Right_Little_1: child Right_Little_Basecover -> Right_Little_Phaprox; limit lower=-0.50 upper=1.4 effort=1000 velocity=3.14 -> lower=0.0872665 upper=1.48353 effort=1.15 velocity=3.14; origin xyz=0.000971571 -0.0433963 0.093583545 rpy=-2.967060 -1.570796 0.000000 -> xyz=0 0 0  rpy=1.5708 0 0; parent base_link -> Right_Little_Basecover
- joint Right_Little_2: child Right_Little_Phoaprox -> Right_Little_Phamed; limit lower=-0.50 upper=1.4 effort=1000 velocity=3.14 -> lower=0.0872665 upper=1.13446 effort=0.6 velocity=3.14; origin xyz=0 0 0  rpy=1.5708 0 0 -> xyz=0.055 0 0 rpy=0 0 0; parent Right_Little_Basecover -> Right_Little_Phaprox
- joint Right_Little_3: child Right_Little_Phamed -> Right_Little_Phadist; limit lower=-0.50 upper=1.4 effort=1000 velocity=3.14 -> lower=0.0872665 upper=1.13446 effort=0.35 velocity=3.14; origin xyz=0.055 0 0 rpy=0 0 0 -> xyz=0.025 0 0 rpy=0 0 -1.570796; parent Right_Little_Phoaprox -> Right_Little_Phamed
- joint Right_Middle_1: child Right_Middle_Basecover -> Right_Middle_Phaprox; limit lower=-0.50 upper=1.4 effort=1000 velocity=3.14 -> lower=0.0872665 upper=1.48353 effort=1.15 velocity=3.14; origin xyz=-0.0037 0.01  0.117783545 rpy=-3.141593 -1.570796 0.000000 -> xyz=0 0 0  rpy=1.5708 0 0; parent base_link -> Right_Middle_Basecover
- joint Right_Middle_2: child Right_Middle_Phoaprox -> Right_Middle_Phamed; limit lower=-0.50 upper=1.4 effort=1000 velocity=3.14 -> lower=0.0872665 upper=1.13446 effort=0.6 velocity=3.14; origin xyz=0 0 0  rpy=1.5708 0 0 -> xyz=0.055 0 0 rpy=0 0 0; parent Right_Middle_Basecover -> Right_Middle_Phaprox
- joint Right_Middle_3: child Right_Middle_Phamed -> Right_Middle_Phadist; limit lower=-0.50 upper=1.4 effort=1000 velocity=3.14 -> lower=0.0872665 upper=1.13446 effort=0.35 velocity=3.14; origin xyz=0.055 0 0 rpy=0 0 0 -> xyz=0.025 0 0 rpy=0 0 -1.570796; parent Right_Middle_Phoaprox -> Right_Middle_Phamed
- joint Right_Ring_1: child Right_Ring_Basecover -> Right_Ring_Phaprox; limit lower=-0.50 upper=1.4 effort=1000 velocity=3.14 -> lower=0.0872665 upper=1.48353 effort=1.15 velocity=3.14; origin xyz=0 -0.01680013 0.11258354 rpy=-3.054326 -1.570796 0.000000 -> xyz=0 0 0  rpy=1.5708 0 0; parent base_link -> Right_Ring_Basecover
- joint Right_Ring_2: child Right_Ring_Phoaprox -> Right_Ring_Phamed; limit lower=-0.50 upper=1.4 effort=1000 velocity=3.14 -> lower=0.0872665 upper=1.13446 effort=0.6 velocity=3.14; origin xyz=0 0 0  rpy=1.5708 0 0 -> xyz=0.055 0 0 rpy=0 0 0; parent Right_Ring_Basecover -> Right_Ring_Phaprox
- joint Right_Ring_3: child Right_Ring_Phamed -> Right_Ring_Phadist; limit lower=-0.50 upper=1.4 effort=1000 velocity=3.14 -> lower=0.0872665 upper=1.13446 effort=0.35 velocity=3.14; origin xyz=0.055 0 0 rpy=0 0 0 -> xyz=0.025 0 0 rpy=0 0 -1.570796; parent Right_Ring_Phoaprox -> Right_Ring_Phamed
- joint Right_Thumb_1: child Right_Thumb_Basecover -> Right_Thumb_Phaprox; limit lower=-0.50 upper=1.4 effort=1000 velocity=3.14 -> lower=0.0872665 upper=1.48353 effort=1.15 velocity=3.14; origin xyz=0.06217593 0.044372912 0.078734808 rpy=0.225810 -1.083656 0.411355 -> xyz=0 0 0  rpy=1.5708 0 0; parent base_link -> Right_Thumb_Basecover
- joint Right_Thumb_2: child Right_Thumb_Phoaprox -> Right_Thumb_Phamed; limit lower=-0.50 upper=1.4 effort=1000 velocity=3.14 -> lower=0.0872665 upper=1.13446 effort=0.6 velocity=3.14; origin xyz=0 0 0  rpy=1.5708 0 0 -> xyz=0.055 0 0 rpy=0 0 0; parent Right_Thumb_Basecover -> Right_Thumb_Phaprox
- joint Right_Thumb_3: child Right_Thumb_Phamed -> Right_Thumb_Phadist; limit lower=-0.50 upper=1.4 effort=1000 velocity=3.14 -> lower=0.0872665 upper=1.13446 effort=0.35 velocity=3.14; origin xyz=0.055 0 0 rpy=0 0 0 -> xyz=0.025 0 0 rpy=0 0 -1.570796; parent Right_Thumb_Phoaprox -> Right_Thumb_Phamed
- joint fixed: child base_link -> base_link_hithand; origin (none) -> xyz=0 0 0.1 rpy=0 0 0

Commit message: updated hithand.urdf to include meshes. Needs symlink from mesh folder to Models folder

File: Models/hithand/hithand.urdf (robot description, URDF)
Before this commit: robot hithand, 23 links, 22 joints
Links:
- link Right_Index_Basecover: geometry collision cylinder length=0.001 radius=0.001; visual mesh filename=meshes/visual/finger/hit-hand-2-finger-basecover.dae
- link Right_Index_Phadist: geometry collision mesh filename=meshes/collision/finger/hit-hand-2-finger-phadist.dae; visual mesh filename=meshes/visual/finger/hit-hand-2-finger-phadist.dae
- link Right_Index_Phamed: geometry collision mesh filename=meshes/collision/finger/hit-hand-2-finger-phamed.dae; visual mesh filename=meshes/visual/finger/hit-hand-2-finger-phamed.dae
- link Right_Index_Phaprox: geometry collision mesh filename=meshes/collision/finger/hit-hand-2-finger-phaprox.dae; visual mesh filename=meshes/visual/finger/hit-hand-2-finger-phaprox.dae
- link Right_Little_Basecover: geometry collision cylinder length=0.001 radius=0.001; visual mesh filename=meshes/visual/finger/hit-hand-2-finger-basecover.dae
- link Right_Little_Phadist: geometry collision mesh filename=meshes/collision/finger/hit-hand-2-finger-phadist.dae; visual mesh filename=meshes/visual/finger/hit-hand-2-finger-phadist.dae
- link Right_Little_Phamed: geometry collision mesh filename=meshes/collision/finger/hit-hand-2-finger-phamed.dae; visual mesh filename=meshes/visual/finger/hit-hand-2-finger-phamed.dae
- link Right_Little_Phaprox: geometry collision mesh filename=meshes/collision/finger/hit-hand-2-finger-phaprox.dae; visual mesh filename=meshes/visual/finger/hit-hand-2-finger-phaprox.dae
- link Right_Middle_Basecover: geometry collision cylinder length=0.001 radius=0.001; visual mesh filename=meshes/visual/finger/hit-hand-2-finger-basecover.dae
- link Right_Middle_Phadist: geometry collision mesh filename=meshes/collision/finger/hit-hand-2-finger-phadist.dae; visual mesh filename=meshes/visual/finger/hit-hand-2-finger-phadist.dae
- link Right_Middle_Phamed: geometry collision mesh filename=meshes/collision/finger/hit-hand-2-finger-phamed.dae; visual mesh filename=meshes/visual/finger/hit-hand-2-finger-phamed.dae
- link Right_Middle_Phaprox: geometry collision mesh filename=meshes/collision/finger/hit-hand-2-finger-phaprox.dae; visual mesh filename=meshes/visual/finger/hit-hand-2-finger-phaprox.dae
- link Right_Ring_Basecover: geometry collision cylinder length=0.001 radius=0.001; visual mesh filename=meshes/visual/finger/hit-hand-2-finger-basecover.dae
- link Right_Ring_Phadist: geometry collision mesh filename=meshes/collision/finger/hit-hand-2-finger-phadist.dae; visual mesh filename=meshes/visual/finger/hit-hand-2-finger-phadist.dae
- link Right_Ring_Phamed: geometry collision mesh filename=meshes/collision/finger/hit-hand-2-finger-phamed.dae; visual mesh filename=meshes/visual/finger/hit-hand-2-finger-phamed.dae
- link Right_Ring_Phaprox: geometry collision mesh filename=meshes/collision/finger/hit-hand-2-finger-phaprox.dae; visual mesh filename=meshes/visual/finger/hit-hand-2-finger-phaprox.dae
- link Right_Thumb_Basecover: geometry collision cylinder length=0.001 radius=0.001; visual mesh filename=meshes/visual/finger/hit-hand-2-finger-basecover.dae
- link Right_Thumb_Phadist: geometry collision mesh filename=meshes/collision/finger/hit-hand-2-finger-phadist.dae; visual mesh filename=meshes/visual/finger/hit-hand-2-finger-phadist.dae
- link Right_Thumb_Phamed: geometry collision mesh filename=meshes/collision/finger/hit-hand-2-finger-phamed.dae; visual mesh filename=meshes/visual/finger/hit-hand-2-finger-phamed.dae
- link Right_Thumb_Phaprox: geometry collision mesh filename=meshes/collision/finger/hit-hand-2-finger-phaprox.dae; visual mesh filename=meshes/visual/finger/hit-hand-2-finger-phaprox.dae
- link base_link_hithand: geometry collision mesh filename=meshes/collision/palm/hit-hand-2-palm-right-merged.dae; visual mesh filename=meshes/visual/palm/hit-hand-2-palm-right.dae
